File: production/ecad/Sensify Main Board/Haptics.kicad_sch (KiCad schematic)
At the start: 0 parts

Commit message: started schematic
Parts:
- added C1, C3: 1 uF, symbol Device:C_Small
- added C2: C_Small, symbol Device:C_Small
- added U1: DRV2605LDGSR, DRV2605LDGSR:SOP50P490X110-10N, symbol DRV2605LDGSR:DRV2605LDGSR
- added U2: TPS73633MDBVREP, TPS73633MDBVREP:SOT95P280X145-5N, symbol TPS73633MDBVREP:TPS73633MDBVREP
Connections:
- new net: C1.1, U1.1 (REG)
- new net: C2.1, U2.5 (OUT)
- new net 5.5 V: C3.2, U1.10 (VDD), U2.1 (IN), U2.3 (EN)
- new net EN: U1.5 (EN)
- new net Earth: C1.2, C2.2, C3.1, U1.4 (IN/TRIG), U1.8 (GND), U2.2 (GND)
- new net LRA_OUT1: U1.7 (OUT+)
- new net LRA_OUT2: U1.9 (OUT-)
- new net SCL: U1.2 (SCL)
- new net SDA: U1.3 (SDA)
- no-connect marks 0 -> 2

Commit message: schematic continued
Parts:
- added R10, R11: 2.2 kΩ, symbol Device:R_US
Connections:
- net SCL: now also R10.2
- net SDA: now also R11.2
- net AVCC: now reaches C2.1, U2.5 (OUT)
- net AVCC: now also R10.1, R11.1
Other:
- moved on the sheet: C2, U1, U2

Commit message: updated schematic
Parts:
- added C14: 1 uF, symbol Device:C_Small
- added R12: 9.76 kΩ, symbol Device:R_US
- C2: value C_Small -> 1 uF
Connections:
- net AVCC: now also C14.1, R12.1
- net Earth: now also C14.2
- new net SBWTDIO: R12.2
Changed lines of the file:
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@@
   (junction (at 105.41 85.09) (diameter 0) (color 0 0 0 0)
   )
+  (junction (at 90.17 85.09) (diameter 0) (color 0 0 0 0)
+  )
   (junction (at 214.63 114.3) (diameter 0) (color 0 0 0 0)
   )
   (junction (at 90.17 123.19) (diameter 0) (color 0 0 0 0)
   )
-  (junction (at 90.17 85.09) (diameter 0) (color 0 0 0 0)
+  (junction (at 81.28 85.09) (diameter 0) (color 0 0 0 0)
+  )
+  (junction (at 66.04 85.09) (diameter 0) (color 0 0 0 0)
   )
   (junction (at 119.38 85.09) (diameter 0) (color 0 0 0 0)
@@
     (stroke (width 0) (type default))
   )
+  (wire (pts (xy 66.04 85.09) (xy 66.04 87.63))
+    (stroke (width 0) (type default))
+  )
   (wire (pts (xy 142.24 118.11) (xy 121.92 118.11))
     (stroke (width 0) (type default))
@@
     (stroke (width 0) (type default))
   )
-  (wire (pts (xy 119.38 90.17) (xy 119.38 96.52))
+  (wire (pts (xy 119.38 93.98) (xy 119.38 96.52))
     (stroke (width 0) (type default))
   )
@@
     (stroke (width 0) (type default))
   )
-  (wire (pts (xy 68.58 85.09) (xy 90.17 85.09))
+  (wire (pts (xy 81.28 85.09) (xy 90.17 85.09))
+    (stroke (width 0) (type default))
+  )
+  (wire (pts (xy 50.8 92.71) (xy 50.8 93.98))
     (stroke (width 0) (type default))
   )
@@
     (stroke (width 0) (type default))
   )
+  (wire (pts (xy 90.17 85.09) (xy 90.17 92.71))
+    (stroke (width 0) (type default))
+  )
   (wire (pts (xy 210.82 114.3) (xy 210.82 125.73))
     (stroke (width 0) (type default))
@@
     (stroke (width 0) (type default))
   )
+  (wire (pts (xy 50.8 85.09) (xy 66.04 85.09))
+    (stroke (width 0) (type default))
+  )
   (wire (pts (xy 177.8 125.73) (xy 191.77 125.73))
     (stroke (width 0) (type default))
@@
     (stroke (width 0) (type default))
   )
+  (wire (pts (xy 119.38 88.9) (xy 119.38 85.09))
+    (stroke (width 0) (type default))
+  )
+  (wire (pts (xy 66.04 85.09) (xy 81.28 85.09))
+    (stroke (width 0) (type default))
+  )
   (wire (pts (xy 165.1 64.77) (xy 158.75 64.77))
     (stroke (width 0) (type default))
   )
+  (wire (pts (xy 50.8 85.09) (xy 50.8 87.63))
+    (stroke (width 0) (type default))
+  )
   (wire (pts (xy 138.43 97.79) (xy 210.82 97.79))
     (stroke (width 0) (type default))
@@
     (stroke (width 0) (type default))
   )
+  (wire (pts (xy 81.28 85.09) (xy 81.28 90.17))
+    (stroke (width 0) (type default))
+  )
   (wire (pts (xy 210.82 114.3) (xy 214.63 114.3))
     (stroke (width 0) (type default))
@@
     (stroke (width 0) (type default))
   )
+  (wire (pts (xy 66.04 95.25) (xy 66.04 99.06))
+    (stroke (width 0) (type default))
+  )
   (wire (pts (xy 158.75 67.31) (xy 165.1 67.31))
     (stroke (width 0) (type default))
   )
   (wire (pts (xy 158.75 66.04) (xy 151.13 66.04))
-    (stroke (width 0) (type default))
-  )
-  (wire (pts (xy 90.17 85.09) (xy 90.17 92.71))
     (stroke (width 0) (type default))
   )
@@
     (effects (font (size 1.27 1.27)) (justify right))
   )
-  (hierarchical_label "AVCC" (shape input) (at 68.58 85.09 180) (fields_autoplaced)
+  (hierarchical_label "SBWTDIO" (shape input) (at 66.04 99.06 270) (fields_autoplaced)
+    (effects (font (size 1.27 1.27)) (justify right))
+  )
+  (hierarchical_label "AVCC" (shape input) (at 81.28 90.17 270) (fields_autoplaced)
     (effects (font (size 1.27 1.27)) (justify right))
   )
@@
     )
   )
+  (symbol (lib_id "Device:R_US") (at 66.04 91.44 0) (unit 1)
+    (in_bom yes) (on_board yes) (dnp no) (fields_autoplaced)
+    (property "Reference" "R12" (at 68.58 90.17 0)
+      (effects (font (size 1.27 1.27)) (justify left) hide)
+    )
+    (property "Value" "9.76 kΩ" (at 68.58 91.44 0)
+      (effects (font (size 1.27 1.27)) (justify left))
+    )
+    (property "Footprint" "" (at 67.056 91.694 90)
+      (effects (font (size 1.27 1.27)) hide)
+    )
+    (property "Datasheet" "~" (at 66.04 91.44 0)
+      (effects (font (size 1.27 1.27)) hide)
+    )
+    (pin "1")
+    (pin "2")
+    (instances
+      (project "Sensify Main Board"
+        (path "/9a7ba7c3-7d28-4a83-bdbc-38fbff59fcbe/326628ab-ecd6-4a75-a8ad-db965643b25a"
+          (reference "R12") (unit 1)
+        )
+      )
+    )
+  )
   (symbol (lib_id "power:Earth") (at 205.74 77.47 0) (unit 1)
     (in_bom yes) (on_board yes) (dnp no) (fields_autoplaced)
@@
     )
   )
+  (symbol (lib_id "Device:C_Small") (at 50.8 90.17 0) (unit 1)
+    (in_bom yes) (on_board yes) (dnp no) (fields_autoplaced)
+    (property "Reference" "C14" (at 53.34 88.9063 0)
+      (effects (font (size 1.27 1.27)) (justify left) hide)
+    )
+    (property "Value" "1 uF" (at 53.34 90.1763 0)
+      (effects (font (size 1.27 1.27)) (justify left))
+    )
+    (property "Footprint" "" (at 50.8 90.17 0)
+      (effects (font (size 1.27 1.27)) hide)
+    )
+    (property "Datasheet" "~" (at 50.8 90.17 0)
+      (effects (font (size 1.27 1.27)) hide)
+    )
+    (pin "2")
+    (pin "1")
+    (instances
+      (project "Sensify Main Board"
+        (path "/9a7ba7c3-7d28-4a83-bdbc-38fbff59fcbe/326628ab-ecd6-4a75-a8ad-db965643b25a"
+          (reference "C14") (unit 1)
+        )
+      )
+    )
+  )
   (symbol (lib_id "Device:R_US") (at 90.17 96.52 0) (unit 1)
     (in_bom yes) (on_board yes) (dnp no) (fields_autoplaced)
@@
     )
   )
-  (symbol (lib_id "Device:C_Small") (at 119.38 87.63 0) (unit 1)
-    (in_bom yes) (on_board yes) (dnp no) (fields_autoplaced)
-    (property "Reference" "C2" (at 121.92 86.3663 0)
+  (symbol (lib_id "Device:C_Small") (at 119.38 91.44 0) (unit 1)
+    (in_bom yes) (on_board yes) (dnp no) (fields_autoplaced)
+    (property "Reference" "C2" (at 121.92 90.1763 0)
+      (effects (font (size 1.27 1.27)) (justify left) hide)
+    )
+    (property "Value" "1 uF" (at 121.92 91.4463 0)
       (effects (font (size 1.27 1.27)) (justify left))
     )
-    (property "Value" "C_Small" (at 121.92 88.9063 0)
-      (effects (font (size 1.27 1.27)) (justify left))
-    )
-    (property "Footprint" "" (at 119.38 87.63 0)
-      (effects (font (size 1.27 1.27)) hide)
-    )
-    (property "Datasheet" "~" (at 119.38 87.63 0)
+    (property "Footprint" "" (at 119.38 91.44 0)
+      (effects (font (size 1.27 1.27)) hide)
+    )
+    (property "Datasheet" "~" (at 119.38 91.44 0)
       (effects (font (size 1.27 1.27)) hide)
     )
@@
         )
       )
+    )
+  )
+  (symbol (lib_id "power:Earth") (at 50.8 93.98 0) (unit 1)
+    (in_bom yes) (on_board yes) (dnp no) (fields_autoplaced)
+    (property "Reference" "#PWR017" (at 50.8 100.33 0)
+      (effects (font (size 1.27 1.27)) hide)
+    )
+    (property "Value" "Earth" (at 50.8 97.79 0)
+      (effects (font (size 1.27 1.27)) hide)
+    )
+    (property "Footprint" "" (at 50.8 93.98 0)
+      (effects (font (size 1.27 1.27)) hide)
+    )
+    (property "Datasheet" "~" (at 50.8 93.98 0)
+      (effects (font (size 1.27 1.27)) hide)
+    )
+    (pin "1")
+    (instances
+      (project "Sensify Main Board"
+        (path "/9a7ba7c3-7d28-4a83-bdbc-38fbff59fcbe/326628ab-ecd6-4a75-a8ad-db965643b25a"
+          (reference "#PWR017") (unit 1)
+        )
+      )
