File: production/ecad/Sensify Main Board/Haptics.kicad_sch (KiCad schematic)
At the start: 17 parts, among them J6 Conn_01x02_Socket, J7 Conn_01x02_Socket, J8 Conn_01x02_Socket, J9 Conn_01x02_Socket

Commit message: main board
routed haptics, modified 3.3V supply
Connections:
- net Earth is gone; now on net GND: C?.1, C?.1, C?.1, C?.1, C?.2, C?.2, C?.2, C?.2, U?.4 (IN/TRIG), U?.4 (IN/TRIG), U?.4 (IN/TRIG), U?.4 (IN/TRIG), U?.8 (GND), U?.8 (GND), U?.8 (GND), U?.8 (GND)

Commit message: Added LCSC parts to KiCAD
Parts:
- C? (x8): LCSC (none) -> C87144
- U? (x4): LCSC (none) -> C527464
- renumbered J6 to J5, J7 to J6, J8 to J7, J9 to J8, TP9 to TP19
