File: production/ecad/Sensify Main Board/MCU.kicad_sch (KiCad schematic)
At the start: 27 parts, among them J5 1332645, J6 Conn_01x06_Socket, J7 Conn_01x06_Socket, SW2 SW_Push, SW3 SW_Push, U10 AO3400A, U11 ESP32-WROOM-32E__16MB_, U8 CP2102N-A01-GQFN28, U9 AO3400A

Commit message: added text for inter module conection
Other:
- note added: "for intermodule connections i was thinking these adafruit DIY connectors but they don't have any symbols or footprint, which is annoying but not the end of the world. we were thinking of putting these on a breakout board. we would have two magnetic connectors per module. https://www.digikey.com/en/products/detail/adafruit-industries-llc/5467/16637687 on the back of the breakout board would be htt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"
Changed lines of the file:
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@@
     (effects (font (size 6 6)) (justify left bottom))
+  )
+  (text "for intermodule connections i was thinking these adafruit DIY connectors but they don't have any symbols or footprint, \nwhich is annoying but not the end of the world.\nwe were thinking of putting these on a breakout board. we would have two magnetic connectors per module.  \nhttps://www.digikey.com/en/products/detail/adafruit-industries-llc/5467/16637687\non the back of the breakout board would be\nhttps://www.digikey.com/en/products/detail/molex/0532611271/699104"
+    (at 17.9832 260.0706 0)
+    (effects (font (size 4 4)) (justify left bottom))
   )
   (text "Reset Button for MCU" (at 43.18 25.4 0)

Commit message: "Improved MCU Schematic"
Parts:
- removed J7: Conn_01x06_Socket, symbol Connector:Conn_01x06_Socket
- removed U10, U9: AO3400A, SOT-23-3L_AOS, symbol A03400A:AO3400A
- removed U11: ESP32-WROOM-32E__16MB_, ESP32-WROOM-32E__16MB_:XCVR_ESP32-WROOM-32E__16MB_, symbol ESP32-WROOM-32E:ESP32-WROOM-32E__16MB_
- removed U8: CP2102N-A01-GQFN28, QFN28_5X5_SIL, symbol CP210:CP2102N-A01-GQFN28
- added J4: Conn_01x06_Socket, Connector_Molex:Molex_CLIK-Mate_502382-0670_1x06-1MP_P1.25mm_Vertical, symbol Connector:Conn_01x06_Socket
- added Q4, Q6: AO3400A, Sensify Footprints:SOT95P280X125-3N, symbol A03400A:AO3400A
- added R35, R40, R41: 0, symbol Device:R
- added R36, R37, R38, R47, R48: 0, Resistor_SMD:R_0402_1005Metric, symbol Device:R
- added R44, R45: 4.7k, Resistor_SMD:R_01005_0402Metric, symbol Device:R
- added U7: CP2102N-A02-GQFN28, Sensify Footprints:QFN28_5X5_SIL-M, symbol CP2102N-A02-GQFN28:CP2102N-A02-GQFN28
- added U8: ESP32-WROOM-32E-N16, Sensify Footprints:ESP32-WROOM-32E_EXP, symbol ESP32-WROOM-32E:ESP32-WROOM-32E-N16
- J5: footprint 1332645:PHOENIX_1332645 -> Sensify Footprints:PHOENIX_1332645
- J6: footprint (none) -> Connector_Molex:Molex_CLIK-Mate_502382-0670_1x06-1MP_P1.25mm_Vertical
Connections:
- net +3V3: now also J4.6 (Pin_6), U7.6 (VDD), U7.7 (VREGIN), U8.2 (3V3)
- net +5V: now also J6.6 (Pin_6), R44.1, R45.1; no longer J6.1 (Pin_1)
- net DTR: now also Q6.2, U7.28 (DTR)
- net EN: now also Q4.3, U8.3 (EN)
- net GND: now also J4.5 (Pin_5), U7.29 (GND), U7.3 (GND), U8.1 (GND), U8.15 (GND), U8.38 (GND), U8.39 (GND), U8.40 (GND), U8.41 (GND), U8.42 (GND), U8.43 (GND), U8.44 (GND), U8.45 (GND), U8.46 (GND), U8.47 (GND)
- net INTERRUPT2_IMU: now also U8.23 (IO15)
- net IO0: now also Q6.3, U8.25 (IO0)
- net MCU_WAKEUP: now also U8.24 (IO2)
- net RTS: now also Q4.2, U7.24 (RTS)
- net SCL: now also R44.2, U8.36 (IO22)
- net SDA: now also R45.2, U8.37 (IO23)
- net UART_RXD: now also R40.1
- net UART_TXD: now also R41.1
- net USB_D+: now also U7.4 (D+)
- net USB_D-: now also U7.5 (D-)
- net at R26.1: now also U7.11 (SUSPENDb)
- net at R32.2: now also Q6.1
- net at R12.2: now also U7.9 (RSTb)
- net at R31.2: now also Q4.1
- net at R20.2, R21.1: now also U7.8 (VBUS)
- net at J6.2 (Pin_2): now also U8.13 (IO14)
- net at J6.3 (Pin_3): now also U8.12 (IO27)
- net at J6.4 (Pin_4): now also U8.11 (IO26)
- net at J6.5 (Pin_5): now also U8.10 (IO25)
- net at R28.1: now also U7.25 (RXD)
- net at R27.1: now also U7.26 (TXD)
- net VBUS renamed FLASHING_VBUS
- new net: J6.1 (Pin_1), U8.14 (IO12)
- new net: J4.4 (Pin_4), U8.28 (IO17)
- new net: J4.3 (Pin_3), U8.29 (IO5)
- new net: J4.2 (Pin_2), U8.30 (IO18)
- new net: J4.1 (Pin_1), U8.31 (IO19)
- new net: R35.2, U8.33 (IO21)
- new net: R41.2, U8.34 (RXD0)
- new net: R40.2, U8.35 (TXD0)
- new net: R48.1, U8.4 (SENSOR_VP)
- new net: R47.1, U8.5 (SENSOR_VN)
- new net: R36.1, U8.6 (IO34)
- new net: R37.1, U8.7 (IO35)
- new net: R38.1, U8.8 (IO32)
- new net INTERRUPT1_IMU: U8.16 (IO13)
- no-connect marks 30 -> 34
Other:
- note added: "ESP32 WROOM 32E-N16"
- note added: "INPUTS"
- note added: "POWER"
- note added: "USB to UART BRIDGE"
- note removed: "ESP32 WROOM 32E"
- note removed: "USB to UART"
- moved on the sheet: C12, C13, C20, C21, C22, C23, J5, J6, R12, R20, R21, R26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

Commit message: Added Novel Mechanism Connection
Parts:
- removed J4, J6: Conn_01x06_Socket, Connector_Molex:Molex_CLIK-Mate_502382-0670_1x06-1MP_P1.25mm_Vertical, symbol Connector:Conn_01x06_Socket
- added J7: 0532611271, Sensify Footprints:MOLEX_0532611271, symbol 0532611271:0532611271
- added R39, R42, R43, R46, R49, R50, R51, R52, R53, R54, R55, R56, R57, R58, R59, R60, R61: 0, Resistor_SMD:R_0402_1005Metric, symbol Device:R
Connections:
- net +3V3: now also J7.12
- net +5V: now also J7.1
- net GND: now also J7.10, J7.S1 (SHIELD), J7.S2 (SHIELD__1)
- net USB_D+: now also R54.2, R57.1, R58.2; no longer J5.A6 (DP1), J5.B6 (DP2), U7.4 (D+)
- net USB_D-: now also R55.2, R56.1, R59.2; no longer J5.A7 (DN1), J5.B7 (DN2), U7.5 (D-)
- net at U8.10 (IO25): now also R49.1
- net at U8.11 (IO26): now also R46.1
- net at U8.12 (IO27): now also R43.1
- net at U8.13 (IO14): now also R42.1
- net at U8.14 (IO12): now also R39.1
- net at U8.26 (IO4): now also R61.2
- net at U8.27 (IO16): now also R60.2
- net at U8.28 (IO17): now also R53.2
- net at U8.29 (IO5): now also R52.2
- net at U8.30 (IO18): now also R51.2
- net at U8.31 (IO19): now also R50.2
- new net: J5.B6 (DP2), R57.2
- new net: J5.A6 (DP1), R54.1
- new net: J5.A7 (DN1), R55.1
- new net: J5.B7 (DN2), R56.2
- new net: R58.1, U7.4 (D+)
- new net: R59.1, U7.5 (D-)
- new net 2: J7.2, R50.1
- new net 3: J7.3, R51.1
- new net 4: J7.4, R52.1
- new net 5: J7.5, R53.1
- new net 6: J7.6, R60.1
- new net 7: J7.7, R61.1
- new net 8: J7.8, R49.2
- new net 9: J7.9, R46.2
- new net DETECT: J7.11, R43.2
Other:
- moved on the sheet: C20, C21, R12, R20, R21, R30

Commit message: Added switch footprints for MCU
Parts:
- SW2, SW3: footprint (none) -> Sensify Footprints:SW_1825910-6-4
Connections:
- net FLASHING_VBUS renamed FLASHING_VBUS_5V
Other:
- note added: "Novel Mechanism Connector"
- moved on the sheet: C12, C13, C20, C21, J7, R12, R20, R21, R26, R27, R28, R35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

Commit message: Improved MCU Schematic
Parts:
- removed R35: 0, symbol Device:R
- removed R36, R37, R38, R39, R42, R47, R48: 0, Resistor_SMD:R_0402_1005Metric, symbol Device:R
Connections:
- net +3V3: now also R44.1, R45.1
- net +5V: no longer R44.1, R45.1
- net IO14: now reaches U8.13 (IO14)
- net IO12: now reaches U8.14 (IO12)
- net IO21: now reaches U8.33 (IO21)
- net IO34: now reaches U8.6 (IO34)
- net IO35: now reaches U8.7 (IO35)
- net IO32: now reaches U8.8 (IO32)
- net IO33: now reaches U8.9 (IO33)
- no-connect marks 34 -> 27
Other:
- moved on the sheet: R40, R41, R43, R44, R45, R46, R49, R50, R51, R52, R53, R60

Commit message: Finished Root Directory for IMU and Haptics
Parts:
- removed R43, R46, R49, R50, R51, R52, R53, R60, R61: 0, Resistor_SMD:R_0402_1005Metric, symbol Device:R
- added J6: Screw_Terminal_01x09, symbol Connector:Screw_Terminal_01x09
- added TP6, TP7, TP8: TestPoint, symbol Connector:TestPoint
Connections:
- net 2 is gone; now on net NovelMechPin2: J7.2
- net 3 is gone; now on net NovelMechPin3: J7.3
- net 4 is gone; now on net NovelMechPin4: J7.4
- net 5 is gone; now on net NovelMechPin5: J7.5
- net 6 is gone; now on net NovelMechPin6: J7.6
- net 8 is gone; now on net NovelMechPin8: J7.8
- net 9 is gone; now on net NovelMechPin9: J7.9
- net DETECT is gone; now on net NovelDetect: J7.11
- net +3V3: now also J6.9 (Pin_9)
- net 7: no longer J7.7
- net EN: now also TP7.1
- net FLASHING_VBUS_5V: now also TP8.1
- net GND: now also J6.1 (Pin_1)
- net IO0: now also TP6.1
- net IO12: now also J6.4 (Pin_4)
- net IO14: now also J6.3 (Pin_3)
- net IO21: now also J6.2 (Pin_2)
- net IO32: now also J6.7 (Pin_7)
- net IO33: now also J6.8 (Pin_8)
- net IO34: now also J6.5 (Pin_5)
- net IO35: now also J6.6 (Pin_6)
- net NovelMechPin8: now reaches U8.10 (IO25)
- net NovelMechPin9: now reaches U8.11 (IO26)
- net NovelDetect: now reaches U8.12 (IO27)
- net NovelMechPin7: now reaches U8.26 (IO4)
- net NovelMechPin7: now also J7.7
- net NovelMechPin6: now reaches U8.27 (IO16)
- net NovelMechPin5: now reaches U8.28 (IO17)
- net NovelMechPin4: now reaches U8.29 (IO5)
- net NovelMechPin3: now reaches U8.30 (IO18)
- net NovelMechPin2: now reaches U8.31 (IO19)
Other:
- note added: "EXTRA GPIO"
- note added: "TEST POINTS"
- note added: "USB to UART"
- note removed: "USB to UART BRIDGE"
- moved on the sheet: C12, C13, J7, R40, R41, R44, R45, U8

Commit message: Finished IMU, Haptics, MCU, and Root Page
Parts:
- removed J6: Screw_Terminal_01x09, symbol Connector:Screw_Terminal_01x09
- added J6: Screw_Terminal_01x08, symbol Connector:Screw_Terminal_01x08
Connections:
- net +3V3: now also J6.8 (Pin_8)
- net GND: now also J6.1 (Pin_1)
- net IO12: now also J6.3 (Pin_3)
- net IO14: now also J6.2 (Pin_2)
- net IO32: now also J6.6 (Pin_6)
- net IO33: now also J6.7 (Pin_7)
- net IO34: now also J6.4 (Pin_4)
- net IO35: now also J6.5 (Pin_5)
- net IO21 renamed HAPTICS_EN
Changed lines of the file:
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@@
+    (stroke (width 0) (type default))
+  )
+  (wire (pts (xy 378.46 152.4) (xy 378.46 153.67))
     (stroke (width 0) (type default))
   )
@@
     (stroke (width 0) (type default))
   )
+  (wire (pts (xy 361.95 100.33) (xy 375.92 100.33))
+    (stroke (width 0) (type default))
+  )
   (wire (pts (xy 121.92 90.17) (xy 121.92 92.71))
     (stroke (width 0) (type default))
@@
     (stroke (width 0) (type default))
   )
-  (wire (pts (xy 378.46 154.94) (xy 367.03 154.94))
+  (wire (pts (xy 378.46 152.4) (xy 367.03 152.4))
     (stroke (width 0) (type default))
   )
@@
     )
   )
-  (global_label "IO21" (shape bidirectional) (at 367.03 152.4 0) (fields_autoplaced)
-    (effects (font (size 1.27 1.27)) (justify left))
-    (property "Intersheetrefs" "${INTERSHEET_REFS}" (at 375.4808 152.4 0)
-      (effects (font (size 1.27 1.27)) (justify left) hide)
-    )
-  )
   (global_label "USB_D-" (shape output) (at 113.03 142.24 0) (fields_autoplaced)
     (effects (font (size 1.27 1.27)) (justify left))
@@
     )
   )
+  (global_label "HAPTICS_EN" (shape input) (at 361.95 100.33 180) (fields_autoplaced)
+    (effects (font (size 1.27 1.27)) (justify right))
+    (property "Intersheetrefs" "${INTERSHEET_REFS}" (at 347.7767 100.33 0)
+      (effects (font (size 1.27 1.27)) (justify right) hide)
+    )
+  )
   (global_label "IO32" (shape bidirectional) (at 193.04 177.8 180) (fields_autoplaced)
     (effects (font (size 1.27 1.27)) (justify right))
@@
     )
   )
-  (global_label "IO21" (shape bidirectional) (at 243.84 195.58 0) (fields_autoplaced)
-    (effects (font (size 1.27 1.27)) (justify left))
-    (property "Intersheetrefs" "${INTERSHEET_REFS}" (at 252.2908 195.58 0)
-      (effects (font (size 1.27 1.27)) (justify left) hide)
-    )
-  )
   (global_label "USB_D+" (shape output) (at 113.03 144.78 0) (fields_autoplaced)
     (effects (font (size 1.27 1.27)) (justify left))
@@
     )
   )
+  (global_label "HAPTICS_EN" (shape input) (at 243.84 195.58 0) (fields_autoplaced)
+    (effects (font (size 1.27 1.27)) (justify left))
+    (property "Intersheetrefs" "${INTERSHEET_REFS}" (at 258.0133 195.58 0)
+      (effects (font (size 1.27 1.27)) (justify left) hide)
+    )
+  )
   (global_label "IO0" (shape input) (at 243.84 215.9 0) (fields_autoplaced)
     (effects (font (size 1.27 1.27)) (justify left))
@@
   )
   (hierarchical_label "SDA" (shape bidirectional) (at 375.92 88.9 0) (fields_autoplaced)
+    (effects (font (size 1.27 1.27)) (justify left))
+  )
+  (hierarchical_label "HAPTICS_EN" (shape input) (at 375.92 100.33 0) (fields_autoplaced)
     (effects (font (size 1.27 1.27)) (justify left))
   )
@@
     )
   )
-  (symbol (lib_id "Connector:Screw_Terminal_01x09") (at 361.95 144.78 180) (unit 1)
-    (in_bom yes) (on_board yes) (dnp no) (fields_autoplaced)
-    (property "Reference" "J6" (at 361.95 128.27 0)
-      (effects (font (size 1.27 1.27)))
-    )
-    (property "Value" "Screw_Terminal_01x09" (at 361.95 130.81 0)
-      (effects (font (size 1.27 1.27)))
-    )
-    (property "Footprint" "" (at 361.95 144.78 0)
-      (effects (font (size 1.27 1.27)) hide)
-    )
-    (property "Datasheet" "~" (at 361.95 144.78 0)
-      (effects (font (size 1.27 1.27)) hide)
-    )
-    (pin "2")
-    (pin "5")
-    (pin "4")
-    (pin "1")
-    (pin "8")
-    (pin "9")
-    (pin "6")
-    (pin "7")
-    (pin "3")
-    (instances
-      (project "Sensify Main Board"
-        (path "/9a7ba7c3-7d28-4a83-bdbc-38fbff59fcbe/ec3ae12c-a69a-4cda-a73d-a33c865c767e"
-          (reference "J6") (unit 1)
-        )
-      )
-    )
-  )
   (symbol (lib_id "Device:C") (at 185.42 57.15 90) (unit 1)
     (in_bom yes) (on_board yes) (dnp no) (fields_autoplaced)
@@
         (path "/9a7ba7c3-7d28-4a83-bdbc-38fbff59fcbe/ec3ae12c-a69a-4cda-a73d-a33c865c767e"
           (reference "R12") (unit 1)
+        )
+      )
+    )
+  )
+  (symbol (lib_id "Connector:Screw_Terminal_01x08") (at 361.95 144.78 180) (unit 1)
+    (in_bom yes) (on_board yes) (dnp no) (fields_autoplaced)
+    (property "Reference" "J6" (at 361.95 128.27 0)
+      (effects (font (size 1.27 1.27)))
+    )
+    (property "Value" "Screw_Terminal_01x08" (at 361.95 130.81 0)
+      (effects (font (size 1.27 1.27)))
+    )
+    (property "Footprint" "" (at 361.95 144.78 0)
+      (effects (font (size 1.27 1.27)) hide)
+    )
+    (property "Datasheet" "~" (at 361.95 144.78 0)
+      (effects (font (size 1.27 1.27)) hide)
+    )
+    (pin "2")
+    (pin "4")
+    (pin "3")
+    (pin "6")
+    (pin "7")
+    (pin "8")
+    (pin "5")
+    (pin "1")
+    (instances
+      (project "Sensify Main Board"
+        (path "/9a7ba7c3-7d28-4a83-bdbc-38fbff59fcbe/ec3ae12c-a69a-4cda-a73d-a33c865c767e"
+          (reference "J6") (unit 1)
         )
       )
@@
     )
   )
-  (symbol (lib_id "power:GND") (at 378.46 154.94 0) (unit 1)
-    (in_bom yes) (on_board yes) (dnp no) (fields_autoplaced)
-    (property "Reference" "#PWR083" (at 378.46 161.29 0)
-      (effects (font (size 1.27 1.27)) hide)
-    )
-    (property "Value" "GND" (at 378.46 160.02 0)
-      (effects (font (size 1.27 1.27)))
-    )
-    (property "Footprint" "" (at 378.46 154.94 0)
-      (effects (font (size 1.27 1.27)) hide)
-    )
-    (property "Datasheet" "" (at 378.46 154.94 0)
-      (effects (font (size 1.27 1.27)) hide)
-    )
+  (symbol (lib_id "power:GND") (at 378.46 153.67 0) (unit 1)
+    (in_bom yes) (on_board yes) (dnp no) (fields_autoplaced)
+    (property "Reference" "#PWR083" (at 378.46 160.02 0)
+      (effects (font (size 1.27 1.27)) hide)
+    )
+    (property "Value" "GND" (at 378.46 158.75 0)
+      (effects (font (size 1.27 1.27)))
+    )
+    (property "Footprint" "" (at 378.46 153.67 0)
+      (effects (font (size 1.27 1.27)) hide)
+    )
+    (property "Datasheet" "" (at 378.46 153.67 0)
+      (effects (font (size 1.27 1.27)) hide)
+    )

Commit message: Added Test Point footprints, fixed Haptics footprints, fixed IMU footprints
Parts:
- J6: footprint (none) -> Connector_PinHeader_2.54mm:PinHeader_1x08_P2.54mm_Vertical
- TP6: footprint (none) -> TestPoint:TestPoint_Pad_D2.0mm
- TP7: renamed from TP8; footprint (none) -> TestPoint:TestPoint_Pad_D2.0mm
- TP8: renamed from TP7; footprint (none) -> TestPoint:TestPoint_Pad_D2.0mm
- renumbered C22 to C27, C23 to C28, C12 to C29, C13 to C30, C20 to C31, C21 to C32, J5 to J4, J7 to J5, Q4 to Q6, Q6 to Q7, R30 to R22, R31 to R23, R32 to R24, R54 to R25, R55 to R26, R56 to R27, R57 to R28, R34 to R30, R33 to R31, R20 to R32, R21 to R33, R12 to R34, R26 to R35, R58 to R36, R59 to R37, R45 to R38, R44 to R39, R27 to R42, R28 to R43, SW3 to SW2, SW2 to SW3, U8 to U5, U7 to U6
