File: production/ecad/Sensify Main Board/BMS.kicad_sch (KiCad schematic)
At the start: 69 parts, among them J1 Screw_Terminal_01x03, J2 Screw_Terminal_01x02, J3 Screw_Terminal_01x03, Q1 NMOS, Q2 NMOS, Q3 NMOS, Q5 NMOS, Q8 PMOS, SW1 SW_Push, U1 MAX17320G22, U2 LD29150DT33R, U4 BQ25306RTER, U6 LM61480Q5RPHRQ1

Commit message: v1 bms ic without charging while using functionality + changed bms hierarchical net labels
Parts:
- removed C1: 0.47u, symbol Device:C
- removed C11: 10u, symbol Device:C_Polarized
- removed C14, C30: 10u, symbol Device:C
- removed C32: 1u, symbol Device:C
- removed C33, C35: 100n, symbol Device:C
- removed C34: 18p, symbol Device:C
- removed C36: 100u, symbol Device:C
- removed D4, D5, D6: D, symbol Device:D
- removed J1, J3: Screw_Terminal_01x03, symbol Connector:Screw_Terminal_01x03
- removed J2: Screw_Terminal_01x02, symbol Connector:Screw_Terminal_01x02
- removed L3: 6.8u, symbol Device:L
- removed Q1, Q2, Q5: NMOS, symbol Simulation_SPICE:NMOS
- removed Q8: PMOS, symbol Simulation_SPICE:PMOS
- removed R10: 100k, symbol Device:R_US
- removed SW1: SW_Push, symbol Switch:SW_Push
- removed TH2: 10k, symbol Device:Thermistor_US
- removed U6: LM61480Q5RPHRQ1, BMS:RPH0016A, symbol BMS:LM61480Q5RPHRQ1
- added 3.3V_TP, 5V_TP, BAT1+_TP, BAT1-/BAT2+1_TP, BAT2-_TP, BMS_ALERT_TP, CHG_TP, DIS_TP1, GND_TP, PACK+_TP, PMID_TP, TH1_TP, USB_9V+: TestPoint, TestPoint:TestPoint_Pad_D1.5mm, symbol Connector:TestPoint
- added C11: 10u, Sensify Footprints:T491A, symbol Device:C_Polarized_US
- added C24: 10u, Capacitor_SMD:C_0805_2012Metric_Pad1.18x1.45mm_HandSolder, symbol Device:C
- added C25: 100u, Sensify Footprints:CAPPM3528X210N, symbol Device:C_Polarized_US
- added C26: 1u, Capacitor_SMD:C_0603_1608Metric_Pad1.08x0.95mm_HandSolder, symbol Device:C
- added C27: 10n, Capacitor_SMD:C_0603_1608Metric_Pad1.08x0.95mm_HandSolder, symbol Device:C
- added C30: 22u, Sensify Footprints:CAPPM3528X210N, symbol Device:C_Polarized_US
- added D1: SK36A-LTP, Sensify Footprints:DIOM5225X244N, symbol Device:D_Schottky
- added D3: CL-196HR-CD-T, Diode_SMD:D_0603_1608Metric_Pad1.05x0.95mm_HandSolder, symbol Device:LED
- added J1: 1-2834011-2, https://www.te.com/commerce/DocumentDelivery/DDEController?Action=srchrtrv&DocNm=1-1773872-7_ModularScrewlessTerminalBl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, symbol Connector_Generic:Conn_01x02
- added J2: 1-2834011-3, symbol Connector_Generic:Conn_01x03
- added L2: 10u, Sensify Footprints:IND_VLS6045EX-100M, symbol Device:L
- added Q1, Q2: PMPB13XNE,115, Sensify Footprints:DFN2020MD-6_SOT1220_NEX, symbol Device:Q_Dual_NMOS_S1G1S2G2D2D2D1D1
- added Q5: BSS223PWH6327XTSA1, symbol Simulation_SPICE:PMOS
- added R35: 150, Resistor_SMD:R_0402_1005Metric_Pad0.72x0.64mm_HandSolder, symbol Device:R_US
- added R36: 100k, Resistor_SMD:R_0402_1005Metric_Pad0.72x0.64mm_HandSolder, symbol Device:R_US
- added R37: 365, Resistor_SMD:R_0402_1005Metric_Pad0.72x0.64mm_HandSolder, symbol Device:R_US
- added R38: 0, Resistor_SMD:R_0402_1005Metric_Pad0.72x0.64mm_HandSolder, symbol Device:R_US
- added S1: PTS_647_SM38_SMTR2_LFS, PTS_647_SM38_SMTR2_LFS:SW_PTS_647_SM38_SMTR2_LFS, symbol BMS:PTS_647_SM38_SMTR2_LFS
- added STAT_TP: TestPoint, TestPoint:TestPoint_Pad_D1.5mm, symbol Connector:TestPoint_Small
- added U6: LM22676MRX-5.0_NOPB, LM22676MRX-5.0_NOPB:VREG_LM5017MR_NOPB, symbol BMS:LM22676MRX-5.0_NOPB
- C18: footprint (none) -> Capacitor_SMD:C_0805_2012Metric_Pad1.18x1.45mm_HandSolder
- C19, C7, C8, C9: footprint (none) -> Capacitor_SMD:C_0402_1005Metric_Pad0.74x0.62mm_HandSolder
- C28: value 10u -> 1u; footprint (none) -> Capacitor_SMD:C_0603_1608Metric_Pad1.08x0.95mm_HandSolder; Material (none) -> CER
- C29: footprint (none) -> Capacitor_SMD:C_0603_1608Metric_Pad1.08x0.95mm_HandSolder; Material (none) -> CER
- C31: value 1u -> 0.47u; footprint (none) -> Capacitor_SMD:C_0402_1005Metric_Pad0.74x0.62mm_HandSolder; Voltage (none) -> 10V; now not fitted
- C32: renamed from C15; footprint (none) -> Capacitor_SMD:C_0402_1005Metric_Pad0.74x0.62mm_HandSolder
- C33: renamed from C16; footprint (none) -> Capacitor_SMD:C_0603_1608Metric_Pad1.08x0.95mm_HandSolder
- C34: renamed from C17; footprint (none) -> Capacitor_SMD:C_0402_1005Metric_Pad0.74x0.62mm_HandSolder
- C35: renamed from C2; footprint (none) -> Capacitor_SMD:C_0402_1005Metric_Pad0.74x0.62mm_HandSolder
- C36: renamed from C3; footprint (none) -> Capacitor_SMD:C_0402_1005Metric_Pad0.74x0.62mm_HandSolder
- C37: renamed from C6; footprint (none) -> Capacitor_SMD:C_0402_1005Metric_Pad0.74x0.62mm_HandSolder
- C38: renamed from C5; footprint (none) -> Capacitor_SMD:C_0402_1005Metric_Pad0.74x0.62mm_HandSolder
- C39: renamed from C4; footprint (none) -> Capacitor_SMD:C_0402_1005Metric_Pad0.74x0.62mm_HandSolder
- D2: footprint (none) -> Diode_SMD:D_0603_1608Metric_Pad1.05x0.95mm_HandSolder; Part number (none) -> LTST-C190GKT
- F1: footprint BMS:ITV4030_LTF -> Sensify Footprints:ITV4030_LTF
- L1: footprint (none) -> Sensify Footprints:IND_PA4332.222NLT_PUL; part number (none) -> PA4332.222NLT
- Q3: value NMOS -> 2N700; footprint (none) -> Sensify Footprints:SOT95P240X111-3N
- R1: footprint (none) -> Sensify Footprints:PS0612_2-10mOHM_YAG; Part number (none) -> PS0612FKF070R005L
- R13: value 1k -> 2.2k; footprint (none) -> Resistor_SMD:R_0402_1005Metric_Pad0.72x0.64mm_HandSolder
- R14: value 33k -> 27k; footprint (none) -> Resistor_SMD:R_0402_1005Metric_Pad0.72x0.64mm_HandSolder; Part number (none) -> ERA-2ARB273X
- R15, R16, R2, R3, R4, R5, R6: footprint (none) -> Resistor_SMD:R_0402_1005Metric_Pad0.72x0.64mm_HandSolder
- R17: value 100k -> 51k; footprint (none) -> Resistor_SMD:R_0603_1608Metric_Pad0.98x0.95mm_HandSolder
- R18: value 4.7k -> 10k; footprint (none) -> Resistor_SMD:R_0402_1005Metric_Pad0.72x0.64mm_HandSolder
- R19: value 24.3k -> 10k; footprint (none) -> Resistor_SMD:R_0402_1005Metric_Pad0.72x0.64mm_HandSolder
- R22: value 100k -> 20k; footprint (none) -> Resistor_SMD:R_0603_1608Metric_Pad0.98x0.95mm_HandSolder
- R23: value 24.9k -> 10k; footprint (none) -> Resistor_SMD:R_0402_1005Metric_Pad0.72x0.64mm_HandSolder
- R24: value 5k -> 0; footprint (none) -> Resistor_SMD:R_0402_1005Metric_Pad0.72x0.64mm_HandSolder; now not fitted
- R25: value 100k -> 0; footprint (none) -> Resistor_SMD:R_0402_1005Metric_Pad0.72x0.64mm_HandSolder; now not fitted
- R7, R8, R9: footprint (none) -> Resistor_SMD:R_0805_2012Metric_Pad1.20x1.40mm_HandSolder
- TH1: Part number (none) -> NCP15XH103F03RC
- U10: renamed from U4; footprint BMS:IC_BQ25306RTER -> Sensify Footprints:IC_BQ25306RTER
- U9: renamed from U1; footprint BMS:TQFN-24 -> Sensify Footprints:TQFN-24
- renumbered U2 to U11
Connections:
- net PACK- is gone; now on net GND: R1.4
- net +3.3V: now also 3.3V_TP.1, C11.1, GND_TP.1, Q5.3 (S), R36.1
- net +5V: now also C28.1, C29.1, 5V_TP.1, C25.1, L2.2, U6.4 (FB); no longer R22.1, R25.1
- net BAT1+: now also BAT1+_TP.1, J2.1 (Pin_1), USB_9V+.1; no longer C18.1, C19.1, L1.2, R15.1, R18.2, R19.1, R2.1, R3.1, U10.10 (BAT), U10.7 (TS)
- net BAT1-/BAT2+: now also BAT1-/BAT2+1_TP.1, J2.2 (Pin_2)
- net GND: now also Q3.3 (S), R22.2, R24.2, U9.EP, U9.P$1 (EP), U9.P$2 (EP), U9.P$3 (EP), U9.P$4 (EP), U9.P$5 (EP), BAT2-_TP.1, C11.2, C24.2, C25.2, C26.2, C30.2, D1.2 (A), D3.1 (K), J1.2 (Pin_2), J2.3 (Pin_3), R38.2, S1.1, U6.6 (GND-1), U6.9 (GND); no longer Q3.1 (D), R17.2
- net USB_9V+: now also J1.1 (Pin_1)
- net at F1.2: now also Q3.1 (D); no longer Q3.3 (S)
- net at U9.7 (ALRT): now also R35.2
- net at C38.1, F1.1: now also Q1.4 (S), Q1.8 (S)
- net at C38.2, R4.1: now also CHG_TP.1, Q1.3 (G)
- net CHARGER_EN: now reaches R25.2
- net CHARGER_EN: now also U10.6 (~{EN}), R38.1
- net at D2.1 (K), R13.2: now also STAT_TP.1
- net at TH1.2, U9.10 (TH1): now also TH1_TP.1
- net AOLDO_OUT: now reaches U9.12 (AOLDO)
- net AOLDO_OUT: now also C31.1, R23.1, R25.1
- net PACK+: now reaches R17.1
- net PACK+: now also C18.1, C19.1, L1.2, R15.1, R2.1, R3.1, U10.10 (BAT), C26.1, C30.1, PACK+_TP.1, Q2.4 (S), Q2.8 (S), U6.7 (VIN)
- net at R5.1: now also DIS_TP1.1, Q2.3 (G)
- net at R24.1: now also U10.5 (POL)
- removed net SYSTEM_POWER: C28.1, C29.1, C31.1, U10.16 (PMID)
- new net: R18.2, R19.1, U10.7 (TS)
- new net: C27.1, U6.1 (BOOT)
- new net: R17.2, R22.1, U6.5 (EN)
- new net: C27.2, D1.1 (K), L2.1, U6.8 (SW)
- new net: Q5.1 (D), R37.1
- new net: D3.2 (A), R37.2
- new net: Q1.1 (D), Q1.2 (D), Q1.5 (D), Q1.6 (D), Q1.7 (D), Q2.1 (D), Q2.2 (D), Q2.5 (D), Q2.6 (D), Q2.7 (D)
- new net: C24.1, PMID_TP.1, U10.16 (PMID)
- new net BMS_ALERT: BMS_ALERT_TP.1, Q5.2 (G), R35.1, R36.2, S1.3
Other:
- note added: "3.3V LDO"
- note added: "Alert indicator LED"
- note added: "BMIC wakeup pushbutton"
- note added: "Batteries"
- note added: "Charge V = 1.1(1+1.33M/200k) = 8.415V"
- note added: "Charge current Ichg = 40k/RIchg 40k/27k = ~1.5A"
- note added: "Charge status LED (Green)"
- note added: "Connectors"
- note added: "Four states: 1. Not charging, system on - batteries power load 2. Charging, system off - charge batteries 3. Charging, system on - disconnect power to load, charge batteries 4. Not charging, not using"
- note added: "I/O"
- note added: "L=(Vin-Vout)*(Vout)/(0.3*Iout*Fsw*Vin) L=(9-5)*(5)/(0.3*1.5*500k*9) = 9.9uH"
- note added: "Power"
- note added: "REnt = REnb*(Voff/Ven-1) REnt = 20k*(5.8/1.6 - 1) ~= 51k"
- note added: "Renb"
- note added: "Rent"
- note added: "Test Points"
- note added: "USB-C 9V+"
- note removed: "103AT-2"
- note removed: "5V->3.3V LDO"
- note removed: "9-8.4V->5V buck(3A) and 5V->3.3V LDO(1.5A)"
- note removed: "Charge V = 1.1(1+1.33M/200k)"
- note removed: "Charge current Ichg = 40k/RIchg ~1.2A = 40k/33k"
- note removed: "Drill"
- note removed: "Either from VBUS or batteries"
- note removed: "External signals"
- note removed: "Haptics"
- note removed: "IMU"
- note removed: "Indicator LED"
- note removed: "MCU"
- note removed: "Main board"
- note removed: "Power ground"
- note removed: "Signal ground"
- note removed: "Vise"
- note removed: "Webench generated"
- note removed: "place to enable ZVC recovery current"
- note removed: "pulldown R unsure"
- moved on the sheet: C10, C18, C19, C32, C33, C34, C35, C36, C37, C38, C39, C7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
