File: production/ecad/Sensify Main Board/BMS.kicad_sch (KiCad schematic)
At the start: 76 parts, among them J1 1-2834011-3, J2 1-2834011-2, Q1 2N700, Q2 PMPB13XNE,115, Q3 PMPB13XNE,115, Q4 BSS223PWH6327XTSA1, Q7 DMP3099L-7, SW1 500ASSP3M2QE, U1 MAX17320G22, U2 BQ25306RTER, U3 LD29150DT33R, U4 LM22676MRX-5.0_NOPB

Commit message: added JLC part numbers to main board
Parts:
- Q1: LCSC (none) -> C8545
- Q4: LCSC (none) -> C3278612
- Q7: LCSC (none) -> C155244
- R1: LCSC (none) -> C103908
- R10: LCSC (none) -> C11896
- R11: LCSC (none) -> C114755
- R12: LCSC (none) -> C226698
- R13, R16, R17, R4: LCSC (none) -> C881209
- R14: LCSC (none) -> C5713265
- R15: LCSC (none) -> C25764
- R18: LCSC (none) -> C25143
- R19: LCSC (none) -> C102750
- R2, R3: LCSC (none) -> C2828807
- R20: LCSC (none) -> C227016
- R21: LCSC (none) -> C95329
- R22: LCSC (none) -> C125934
- R41: LCSC C95329 -> C881209
- R42, R7: LCSC (none) -> C60485
- R6, R8: LCSC (none) -> C102747
- R9: LCSC (none) -> C25933
- TH1: LCSC (none) -> C77131
Changed lines of the file:
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@@
       (effects (font (size 1.27 1.27)) hide)
     )
+    (property "LCSC" "C881209" (at 140.97 241.3 0)
+      (effects (font (size 1.27 1.27)) hide)
+    )
     (pin "1")
     (pin "2")
@@
       (effects (font (size 1.27 1.27)) hide)
     )
+    (property "LCSC" "C155244" (at 236.22 208.28 0)
+      (effects (font (size 1.27 1.27)) hide)
+    )
     (pin "2")
     (pin "1")
@@
       (effects (font (size 1.27 1.27)) hide)
     )
+    (property "LCSC" "C102750" (at 177.8 111.76 0)
+      (effects (font (size 1.27 1.27)) hide)
+    )
     (pin "1")
     (pin "2")
@@
       (effects (font (size 1.27 1.27)) hide)
     )
+    (property "LCSC" "C60485" (at 88.9 220.98 0)
+      (effects (font (size 1.27 1.27)) hide)
+    )
     (pin "1")
     (pin "2")
@@
       (effects (font (size 1.27 1.27)) hide)
     )
+    (property "LCSC" "C881209" (at 140.97 232.41 0)
+      (effects (font (size 1.27 1.27)) hide)
+    )
     (pin "1")
     (pin "2")
@@
       (effects (font (size 1.27 1.27)) hide)
     )
+    (property "LCSC" "C2828807" (at 52.07 124.46 0)
+      (effects (font (size 1.27 1.27)) hide)
+    )
     (pin "1")
     (pin "2")
@@
       (effects (font (size 1.27 1.27)) hide)
     )
+    (property "LCSC" "C25764" (at 138.43 219.71 0)
+      (effects (font (size 1.27 1.27)) hide)
+    )
     (pin "1")
     (pin "2")
@@
       (effects (font (size 1.27 1.27)) hide)
     )
+    (property "LCSC" "C227016" (at 207.01 125.73 0)
+      (effects (font (size 1.27 1.27)) hide)
+    )
     (pin "1")
     (pin "2")
@@
       (effects (font (size 1.27 1.27)) hide)
     )
+    (property "LCSC" "C3278612" (at 204.47 116.84 0)
+      (effects (font (size 1.27 1.27)) hide)
+    )
     (pin "2")
     (pin "1")
@@
       (effects (font (size 1.27 1.27)) hide)
     )
+    (property "LCSC" "C881209" (at 63.5 105.41 0)
+      (effects (font (size 1.27 1.27)) hide)
+    )
     (pin "1")
     (pin "2")
@@
       (effects (font (size 1.27 1.27)) hide)
     )
+    (property "LCSC" "C102747" (at 86.36 97.79 0)
+      (effects (font (size 1.27 1.27)) hide)
+    )
     (pin "1")
     (pin "2")
@@
       (effects (font (size 1.27 1.27)) hide)
     )
+    (property "LCSC" "C8545" (at 55.88 100.33 0)
+      (effects (font (size 1.27 1.27)) hide)
+    )
     (pin "1")
     (pin "2")
@@
       (effects (font (size 1.27 1.27)) hide)
     )
+    (property "LCSC" "C95329" (at 298.45 214.63 0)
+      (effects (font (size 1.27 1.27)) hide)
+    )
     (pin "1")
     (pin "2")
@@
       (effects (font (size 1.27 1.27)) hide)
     )
+    (property "LCSC" "C114755" (at 111.76 105.41 0)
+      (effects (font (size 1.27 1.27)) hide)
+    )
     (pin "1")
     (pin "2")
@@
       (effects (font (size 1.27 1.27)) hide)
     )
+    (property "LCSC" "C25933" (at 92.71 203.2 0)
+      (effects (font (size 1.27 1.27)) hide)
+    )
     (pin "1")
     (pin "2")
@@
       (effects (font (size 1.27 1.27)))
     )
+    (property "LCSC" "C77131" (at 104.14 148.59 0)
+      (effects (font (size 1.27 1.27)) hide)
+    )
     (pin "1")
     (pin "2")
@@
       (effects (font (size 1.27 1.27)) hide)
     )
+    (property "LCSC" "C25143" (at 146.05 116.84 0)
+      (effects (font (size 1.27 1.27)) hide)
+    )
     (pin "1")
     (pin "2")
@@
       (effects (font (size 1.27 1.27)) hide)
     )
-    (property "LCSC" "C95329" (at 228.6 199.39 0)
+    (property "LCSC" "C881209" (at 228.6 199.39 0)
       (effects (font (size 1.27 1.27)) hide)
     )
@@
       (effects (font (size 1.27 1.27)) hide)
     )
+    (property "LCSC" "C11896" (at 92.71 207.01 0)
+      (effects (font (size 1.27 1.27)) hide)
+    )
     (pin "1")
     (pin "2")
@@
       (effects (font (size 1.27 1.27)) hide)
     )
+    (property "LCSC" "C103908" (at 24.13 104.14 0)
+      (effects (font (size 1.27 1.27)) hide)
+    )
     (pin "1")
     (pin "2")
@@
       (effects (font (size 1.27 1.27)) hide)
     )
+    (property "LCSC" "C102747" (at 91.44 97.79 0)
+      (effects (font (size 1.27 1.27)) hide)
+    )
     (pin "1")
     (pin "2")
@@
       (effects (font (size 1.27 1.27)) hide)
     )
+    (property "LCSC" "C2828807" (at 52.07 140.97 0)
+      (effects (font (size 1.27 1.27)) hide)
+    )
     (pin "1")
     (pin "2")
@@
       (effects (font (size 1.27 1.27)) hide)
     )
+    (property "LCSC" "C60485" (at 236.22 222.25 0)
+      (effects (font (size 1.27 1.27)) hide)
+    )
     (pin "1")
     (pin "2")
@@
       (effects (font (size 1.27 1.27)) hide)
     )
+    (property "LCSC" "C226698" (at 119.38 105.41 0)
+      (effects (font (size 1.27 1.27)) hide)
+    )
     (pin "1")
     (pin "2")
@@
       (effects (font (size 1.27 1.27)) hide)
     )
+    (property "LCSC" "C125934" (at 298.45 222.25 0)
+      (effects (font (size 1.27 1.27)) hide)
+    )
     (pin "1")
     (pin "2")
@@
       (effects (font (size 1.27 1.27)) hide)
     )
+    (property "LCSC" "C5713265" (at 138.43 212.09 0)
+      (effects (font (size 1.27 1.27)) hide)
+    )
     (pin "1")
     (pin "2")
@@
       (effects (font (size 1.27 1.27)) hide)
     )
+    (property "LCSC" "C881209" (at 133.35 132.08 0)
+      (effects (font (size 1.27 1.27)) hide)
+    )
