File: production/ecad/Sensify Main Board/Sensify Main Board.kicad_pcb (KiCad board)
At the start: 2 copper layers, 0 parts

Commit message: started main board layout
Parts:
- added BAT1+_TP1: TestPoint, TestPoint:TestPoint_Pad_D1.5mm, F.Cu at (17.2, 33.5)
- added BAT1-/BAT2+_TP1: TestPoint, TestPoint:TestPoint_Pad_D1.5mm, F.Cu at (17.2, 37.0)
- added BAT2-_TP1: TestPoint, TestPoint:TestPoint_Pad_D1.5mm, F.Cu at (17.2, 40.6)
- added BMS_ALERT_TP1: TestPoint, TestPoint:TestPoint_Pad_D1.5mm, F.Cu at (17.2, 44.1)
- added C1: 0.47u, Capacitor_SMD:C_0402_1005Metric_Pad0.74x0.62mm_HandSolder, F.Cu at (118.6, 110.0)
- added C10: 10u, Capacitor_SMD:C_0805_2012Metric_Pad1.18x1.45mm_HandSolder, F.Cu at (33.0, 11.9)
- added C11: 0.01u, Capacitor_SMD:C_0402_1005Metric_Pad0.74x0.62mm_HandSolder, F.Cu at (140.9, 109.0)
- added C12: 47n, Capacitor_SMD:C_0402_1005Metric_Pad0.74x0.62mm_HandSolder, F.Cu at (38.6, 41.7)
- added C13: 0.47u, Capacitor_SMD:C_0402_1005Metric_Pad0.74x0.62mm_HandSolder, F.Cu at (38.6, 43.6)
- added C14: 470p, Capacitor_SMD:C_0402_1005Metric_Pad0.74x0.62mm_HandSolder, F.Cu at (38.6, 45.6)
- added C15: 10u, Capacitor_SMD:C_0805_2012Metric_Pad1.18x1.45mm_HandSolder, F.Cu at (33.0, 14.9)
- added C16: 0.33u, Capacitor_SMD:C_0603_1608Metric_Pad1.08x0.95mm_HandSolder, F.Cu at (1.68, 20.4)
- added C17: 22u, Sensify Footprints:CAPPM3528X210N, F.Cu at (6.97, 40.0)
- added C18: 1u, Capacitor_SMD:C_0603_1608Metric_Pad1.08x0.95mm_HandSolder, F.Cu at (1.68, 22.9)
- added C19: 10u, Sensify Footprints:T491A, F.Cu at (77.2, 22.6)
- added C2: 0.1u, Capacitor_SMD:C_0402_1005Metric_Pad0.74x0.62mm_HandSolder, F.Cu at (141.4, 128.8)
- added C20: 10n, Capacitor_SMD:C_0603_1608Metric_Pad1.08x0.95mm_HandSolder, F.Cu at (1.68, 25.4)
- added C21: 100u, Sensify Footprints:CAPPM3528X210N, F.Cu at (6.97, 44.6)
- added C22: 1u, Capacitor_SMD:C_0603_1608Metric_Pad1.08x0.95mm_HandSolder, F.Cu at (1.68, 27.9)
- added C23: 1u, Capacitor_SMD:C_0603_1608Metric_Pad1.08x0.95mm_HandSolder, F.Cu at (1.68, 30.4)
- added C24: 0.1uF, Capacitor_SMD:C_0402_1005Metric, F.Cu at (39.0, 72.8)
- added C25: 0.1uF, Capacitor_SMD:C_0402_1005Metric, F.Cu at (39.0, 74.8)
- added C26: 0.1uF, Capacitor_SMD:C_0402_1005Metric, F.Cu at (39.0, 76.8)
- added C27: 10uF, Capacitor_SMD:C_0402_1005Metric, F.Cu at (39.0, 78.7)
- added C28: 4.7uF, Capacitor_SMD:C_0402_1005Metric, F.Cu at (39.0, 80.7)
- added C29: 100nF, Capacitor_SMD:C_0402_1005Metric, F.Cu at (39.0, 82.7)
- added C3: 2.2u, Capacitor_SMD:C_0603_1608Metric_Pad1.08x0.95mm_HandSolder, F.Cu at (1.68, 17.9)
- added C30: 1 uF, Capacitor_SMD:C_0402_1005Metric, F.Cu at (63.5, 49.9)
- added C31: 1 uF, Capacitor_SMD:C_0402_1005Metric, F.Cu at (63.5, 51.8)
- added C32: 1 uF, Capacitor_SMD:C_0402_1005Metric, F.Cu at (63.5, 53.8)
- added C33: 1 uF, Capacitor_SMD:C_0402_1005Metric, F.Cu at (63.5, 55.8)
- added C34: 1 uF, Capacitor_SMD:C_0402_1005Metric, F.Cu at (63.5, 57.7)
- added C35: 1 uF, Capacitor_SMD:C_0402_1005Metric, F.Cu at (63.5, 59.7)
- added C36: 1 uF, Capacitor_SMD:C_0402_1005Metric, F.Cu at (63.5, 61.7)
- added C37: 1 uF, Capacitor_SMD:C_0402_1005Metric, F.Cu at (63.5, 63.6)
- added C38: 100n, Capacitor_SMD:C_0402_1005Metric, F.Cu at (59.6, 38.5)
- added C39: 100n, Capacitor_SMD:C_0402_1005Metric, F.Cu at (59.6, 40.5)
- added C4: 0.01u, Capacitor_SMD:C_0402_1005Metric_Pad0.74x0.62mm_HandSolder, F.Cu at (111.2, 129.3)
- added C5: 0.01u, Capacitor_SMD:C_0402_1005Metric_Pad0.74x0.62mm_HandSolder, F.Cu at (111.2, 131.3)
- added C6: 2.2u, Capacitor_SMD:C_0402_1005Metric_Pad0.74x0.62mm_HandSolder, F.Cu at (35.4, 39.7)
- added C7: 0.1u, Capacitor_SMD:C_0402_1005Metric_Pad0.74x0.62mm_HandSolder, F.Cu at (35.4, 41.7)
- added C8: 0.47u, Capacitor_SMD:C_0402_1005Metric_Pad0.74x0.62mm_HandSolder, F.Cu at (140.9, 117.7)
- added C9: 0.47u, Capacitor_SMD:C_0402_1005Metric_Pad0.74x0.62mm_HandSolder, F.Cu at (140.9, 119.6)
- added CHG_TP1: TestPoint, TestPoint:TestPoint_Pad_D1.5mm, F.Cu at (20.8, 33.5)
- added D1: LED, Diode_SMD:D_0603_1608Metric_Pad1.05x0.95mm_HandSolder, F.Cu at (28.3, 33.0)
- added D2: CL-196HR-CD-T, Diode_SMD:D_0603_1608Metric_Pad1.05x0.95mm_HandSolder, F.Cu at (28.3, 35.6)
- added D3: SK36A-LTP, Sensify Footprints:DIOM5225X244N, F.Cu at (45.4, 18.0)
- added DIS_TP1: TestPoint, TestPoint:TestPoint_Pad_D1.5mm, F.Cu at (20.8, 37.0)
- added F1: ITV4030L1412NR, Sensify Footprints:ITV4030_LTF, F.Cu at (119.2, 117.5)
- added H1: MountingHole, MountingHole:MountingHole_3.2mm_M3, F.Cu at (55.2, 3.48)
- added H2: MountingHole, MountingHole:MountingHole_3.2mm_M3, F.Cu at (55.2, 11.4)
- added H3: MountingHole, MountingHole:MountingHole_3.2mm_M3, F.Cu at (55.2, 19.4)
- added H4: MountingHole, MountingHole:MountingHole_3.2mm_M3, F.Cu at (55.2, 27.3)
- added J1: 1-2834011-3, Sensify Footprints:128340113, F.Cu at (124.4, 128.3)
- added J2: 1-2834011-2, Sensify Footprints:128340112, F.Cu at (152.4, 132.1)
- added J3: 1332645, Sensify Footprints:PHOENIX_1332645, F.Cu at (0.65, 85.7)
- added J4: 0532611271, Sensify Footprints:MOLEX_0532611271, F.Cu at (31.4, 53.9)
- added J5: Screw_Terminal_01x08, Connector_PinHeader_2.54mm:PinHeader_1x08_P2.54mm_Vertical, F.Cu at (22.5, 59.1)
- added J6: Conn_01x02_Socket, Connector_JST:JST_EH_B2B-EH-A_1x02_P2.50mm_Vertical, F.Cu at (48.2, 51.5)
- added J7: Conn_01x02_Socket, Connector_JST:JST_EH_B2B-EH-A_1x02_P2.50mm_Vertical, F.Cu at (48.2, 57.3)
- added J8: Conn_01x02_Socket, Connector_JST:JST_EH_B2B-EH-A_1x02_P2.50mm_Vertical, F.Cu at (48.2, 63.2)
- added J9: Conn_01x02_Socket, Connector_JST:JST_EH_B2B-EH-A_1x02_P2.50mm_Vertical, F.Cu at (48.2, 69.0)
- added L1: 2.2u, Sensify Footprints:IND_PA4332.222NLT_PUL, F.Cu at (40.0, 7.08)
- added L2: 10u, Sensify Footprints:IND_VLS6045EX-100M, F.Cu at (44.1, 24.5)
- added PACK+_TP1: TestPoint, TestPoint:TestPoint_Pad_D1.5mm, F.Cu at (20.8, 40.6)
- added PMID_TP1: TestPoint, TestPoint:TestPoint_Pad_D1.5mm, F.Cu at (20.8, 44.1)
- added Q1: 2N700, Sensify Footprints:SOT95P240X111-3N, F.Cu at (128.8, 120.2)
- added Q2: PMPB13XNE,115, Sensify Footprints:DFN2020MD-6_SOT1220_NEX, F.Cu at (125.0, 102.4)
- added Q3: PMPB13XNE,115, Sensify Footprints:DFN2020MD-6_SOT1220_NEX, F.Cu at (136.1, 102.9)
- added Q4: BSS223PWH6327XTSA1, Sensify Footprints:SOT65P210X100-3N, F.Cu at (39.9, 1.38)
- added Q5: AO3400A, Sensify Footprints:SOT95P280X125-3N, F.Cu at (37.7, 59.1)
- added Q6: AO3400A, Sensify Footprints:SOT95P280X125-3N, F.Cu at (37.7, 63.7)
- added R1: 10, Resistor_SMD:R_0805_2012Metric_Pad1.20x1.40mm_HandSolder, F.Cu at (12.5, 39.2)
- added R10: 2.2k, Resistor_SMD:R_0402_1005Metric_Pad0.72x0.64mm_HandSolder, F.Cu at (32.2, 27.6)
- added R11: 27k, Resistor_SMD:R_0402_1005Metric_Pad0.72x0.64mm_HandSolder, F.Cu at (32.2, 29.6)
- added R12: 0, Resistor_SMD:R_0402_1005Metric_Pad0.72x0.64mm_HandSolder, F.Cu at (35.4, 17.6)
- added R13: 250, Resistor_SMD:R_0402_1005Metric_Pad0.72x0.64mm_HandSolder, F.Cu at (35.4, 19.6)
- added R14: 1k, Resistor_SMD:R_0402_1005Metric_Pad0.72x0.64mm_HandSolder, F.Cu at (35.4, 21.6)
- added R15: 10k, Resistor_SMD:R_0402_1005Metric_Pad0.72x0.64mm_HandSolder, F.Cu at (35.4, 23.6)
- added R16: 1.33M, Resistor_SMD:R_0402_1005Metric_Pad0.72x0.64mm_HandSolder, F.Cu at (35.4, 25.6)
- added R17: 200k, Resistor_SMD:R_0402_1005Metric_Pad0.72x0.64mm_HandSolder, F.Cu at (35.4, 27.6)
- added R18: 10k, Resistor_SMD:R_0402_1005Metric_Pad0.72x0.64mm_HandSolder, F.Cu at (35.4, 29.6)
- added R19: 10k, Resistor_SMD:R_0402_1005Metric_Pad0.72x0.64mm_HandSolder, F.Cu at (38.7, 17.6)
- added R2: 0, Resistor_SMD:R_0402_1005Metric_Pad0.72x0.64mm_HandSolder, F.Cu at (32.2, 17.6)
- added R20: 150, Resistor_SMD:R_0402_1005Metric_Pad0.72x0.64mm_HandSolder, F.Cu at (38.7, 19.6)
- added R21: 100k, Resistor_SMD:R_0402_1005Metric_Pad0.72x0.64mm_HandSolder, F.Cu at (38.7, 21.6)
- added R22: 365, Resistor_SMD:R_0402_1005Metric_Pad0.72x0.64mm_HandSolder, F.Cu at (38.7, 23.6)
- added R23: 51k, Resistor_SMD:R_0603_1608Metric_Pad0.98x0.95mm_HandSolder, F.Cu at (1.68, 32.9)
- added R24: 20k, Resistor_SMD:R_0603_1608Metric_Pad0.98x0.95mm_HandSolder, F.Cu at (1.68, 35.4)
- added R25: 5.1k, Resistor_SMD:R_0402_1005Metric, F.Cu at (26.3, 72.8)
- added R26: 10k, Resistor_SMD:R_0402_1005Metric, F.Cu at (26.3, 74.8)
- added R27: 10k, Resistor_SMD:R_0402_1005Metric, F.Cu at (26.3, 76.8)
- added R28: 0, Resistor_SMD:R_0402_1005Metric, F.Cu at (26.3, 78.8)
- added R29: 0, Resistor_SMD:R_0402_1005Metric, F.Cu at (26.3, 80.8)
- added R3: 0, Resistor_SMD:R_0402_1005Metric_Pad0.72x0.64mm_HandSolder, F.Cu at (32.2, 19.6)
- added R30: 0, Resistor_SMD:R_0402_1005Metric, F.Cu at (26.3, 82.8)
- added R31: 0, Resistor_SMD:R_0402_1005Metric, F.Cu at (26.3, 84.8)
- added R32: 5.1k, Resistor_SMD:R_0402_1005Metric, F.Cu at (29.2, 72.8)
- added R33: 1k, Resistor_SMD:R_0402_1005Metric, F.Cu at (29.2, 74.8)
- added R34: 1k, Resistor_SMD:R_0402_1005Metric, F.Cu at (29.2, 76.8)
- added R35: 22.1k, Resistor_SMD:R_0402_1005Metric, F.Cu at (29.2, 78.8)
- added R36: 47.5k, Resistor_SMD:R_0402_1005Metric, F.Cu at (29.2, 80.8)
- added R37: 10k, Resistor_SMD:R_0402_1005Metric, F.Cu at (29.2, 82.8)
- added R38: 10k, Resistor_SMD:R_0402_1005Metric, F.Cu at (29.2, 84.8)
- added R39: 0, Resistor_SMD:R_0402_1005Metric, F.Cu at (32.1, 72.8)
- added R4: 50, Resistor_SMD:R_0805_2012Metric_Pad1.20x1.40mm_HandSolder, F.Cu at (12.5, 42.2)
- added R40: 0, Resistor_SMD:R_0402_1005Metric, F.Cu at (32.1, 74.8)
- added R41: 4.7k, Resistor_SMD:R_01005_0402Metric, F.Cu at (41.5, 57.6)
- added R42: 4.7k, Resistor_SMD:R_01005_0402Metric, F.Cu at (41.5, 59.2)
- added R43: 0, Resistor_SMD:R_01005_0402Metric, F.Cu at (41.5, 60.9)
- added R44: 0, Resistor_SMD:R_01005_0402Metric, F.Cu at (41.5, 62.5)
- added R45: 0, Resistor_SMD:R_0402_1005Metric, F.Cu at (32.1, 76.8)
- added R46: 0, Resistor_SMD:R_0402_1005Metric, F.Cu at (32.1, 78.8)
- added R47: 0, Resistor_SMD:R_0402_1005Metric, F.Cu at (56.7, 38.5)
- added R48: 1k, Resistor_SMD:R_0402_1005Metric, F.Cu at (56.7, 40.5)
- added R5: 50, Resistor_SMD:R_0805_2012Metric_Pad1.20x1.40mm_HandSolder, F.Cu at (12.5, 45.1)
- added R6: 10k, Resistor_SMD:R_0402_1005Metric_Pad0.72x0.64mm_HandSolder, F.Cu at (32.2, 21.6)
- added R7: 5m, Sensify Footprints:PS0612_2-10mOHM_YAG, F.Cu at (28.1, 39.5)
- added R8: 100, Resistor_SMD:R_0402_1005Metric_Pad0.72x0.64mm_HandSolder, F.Cu at (32.2, 23.6)
- added R9: 100, Resistor_SMD:R_0402_1005Metric_Pad0.72x0.64mm_HandSolder, F.Cu at (32.2, 25.6)
- added S1: PTS_647_SM38_SMTR2_LFS, Sensify Footprints:SW_PTS_647_SM38_SMTR2_LFS, F.Cu at (8.80, 34.7)
- added STAT_TP1: TestPoint, TestPoint:TestPoint_Pad_D1.5mm, F.Cu at (24.3, 33.5)
- added SW1: SW_Push, Sensify Footprints:SW_1825910-6-4, F.Cu at (29.9, 60.5)
- added SW2: SW_Push, Sensify Footprints:SW_1825910-6-4, F.Cu at (29.9, 68.1)
- added SW3: ST141D00, Sensify Footprints:SW_ST141D00, F.Cu at (15.8, 8.06)
- added TH1: 10k, Resistor_SMD:R_0402_1005Metric_Pad0.72x0.64mm_HandSolder, F.Cu at (38.7, 25.6)
- added TH1_TP1: TestPoint, TestPoint:TestPoint_Pad_D1.5mm, F.Cu at (24.3, 37.0)
- added TP1: SDA, TestPoint:TestPoint_Pad_D2.0mm, F.Cu at (61.2, 1.52)
- added TP10: INTERRUPT1_IMU, TestPoint:TestPoint_Pad_D2.0mm, F.Cu at (53.2, 35.3)
- added TP11: INTERRUPT2_IMU, TestPoint:TestPoint_Pad_D2.0mm, F.Cu at (53.2, 39.4)
- added TP2: 3.3V, TestPoint:TestPoint_Pad_D2.0mm, F.Cu at (61.2, 5.58)
- added TP3: GND, TestPoint:TestPoint_Pad_D2.0mm, F.Cu at (61.2, 9.62)
- added TP4: SCL, TestPoint:TestPoint_Pad_D2.0mm, F.Cu at (61.2, 13.7)
- added TP5: 5V, TestPoint:TestPoint_Pad_D2.0mm, F.Cu at (61.2, 17.7)
- added TP6: IO0, TestPoint:TestPoint_Pad_D2.0mm, F.Cu at (35.6, 73.9)
- added TP7: FLASHING_VBUS_5V, TestPoint:TestPoint_Pad_D2.0mm, F.Cu at (35.6, 77.9)
- added TP8: EN, TestPoint:TestPoint_Pad_D2.0mm, F.Cu at (35.6, 82.0)
- added TP9: HAPTICS_EN, TestPoint:TestPoint_Pad_D2.0mm, F.Cu at (56.2, 69.1)
- added U1: MAX17320G22, Sensify Footprints:TQFN-24, F.Cu at (130.5, 112.0)
- added U10: DRV2605LDGSR, Sensify Footprints:SOP50P490X110-10N, F.Cu at (58.4, 64.8)
- added U11: LSM6DSOTR, Sensify Footprints:IMU_LSM6DSOTR, F.Cu at (185.2, 35.3)
- added U2: BQ25306RTER, Sensify Footprints:IC_BQ25306RTER, F.Cu at (152.4, 99.1)
- added U3: LD29150DT33R, Sensify Footprints:DPAK456P972X240-3N, F.Cu at (152.4, 111.8)
- added U4: LM22676MRX-5.0_NOPB, Sensify Footprints:VREG_LM5017MR_NOPB, F.Cu at (164.4, 99.7)
- added U5: ESP32-WROOM-32E-N16, Sensify Footprints:ESP32-WROOM-32E_EXP, F.Cu at (165.7, 34.7)
- added U6: CP2102N-A02-GQFN28, Sensify Footprints:QFN28_5X5_SIL-M, F.Cu at (17.9, 92.9)
- added U7: DRV2605LDGSR, Sensify Footprints:SOP50P490X110-10N, F.Cu at (58.4, 51.1)
- added U8: DRV2605LDGSR, Sensify Footprints:SOP50P490X110-10N, F.Cu at (58.4, 55.7)
- added U9: DRV2605LDGSR, Sensify Footprints:SOP50P490X110-10N, F.Cu at (58.4, 60.2)
- added USB_9V+1: TestPoint, TestPoint:TestPoint_Pad_D1.5mm, F.Cu at (24.3, 40.6)
Routing:
- net (no net): vias 0 -> 2
Other:
- copper layers 2 -> 4
