File: production/ecad/Novel Mechanism 1 Board/Novel Mechanism 1 Board.kicad_pcb (KiCad board)
At the start: 2 copper layers, 39 parts, among them J1 Conn_01x02_Socket, J2 Conn_01x02_Socket, J3 Conn_01x02_Socket, J4 0532611271, U1 ADC081C021CIMM/NOPB, U2 ADC081C021CIMM/NOPB, U3 ADC081C021CIMM/NOPB

Commit message: Update Novel Mechanism 1 Board.kicad_pcb
Parts:
- moved R8 6.40 mm to (27.9, 32.0), turned to -90 degrees
- moved C4 5.81 mm to (46.2, 61.2)
- moved C1 5.60 mm to (43.4, 61.2)
- moved R4 5.39 mm to (42.2, 64.5)
- moved U1 5.38 mm to (38.2, 60.5)
- moved U3 4.43 mm to (31.6, 35.6)
- moved TP1 3.92 mm to (25.9, 34.5)
- moved TP4 3.83 mm to (32.0, 64.3)
- moved R3 3.81 mm to (25.5, 38.1)
- moved R1 3.55 mm to (31.8, 59.9)
- moved J4 3.38 mm to (51.3, 44.4)
- moved TP6 3.36 mm to (31.0, 40.4)
- moved J1 3.34 mm to (23.4, 61.7)
- moved TP2 3.08 mm to (24.4, 56.1)
- moved J2 2.95 mm to (23.4, 50.5)
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Routing:
- net +3V3: track 37.1 -> 141.3 mm, vias 7 -> 2
- net INTERRUPT_F2: track 21.9 -> 32.9 mm
- net INTERRUPT_F1: track 23.2 -> 34.0 mm
- net INTERRUPT_LP: track 24.5 -> 32.4 mm
- net FSR_2: track 7.01 -> 13.2 mm
- net LIN_POT: track 11.6 -> 17.7 mm
- net FSR_1: track 6.91 -> 12.4 mm
- net Net-(U2-ADDR0): track 1.87 -> 6.58 mm
- net GND: track 37.1 -> 39.8 mm, vias 13 -> 14
- net Net-(U3-ADDR0): track 1.87 -> 4.31 mm
- net Net-(U1-ADDR0): track 1.98 -> 4.11 mm
- net Net-(U3-ADDR1): track 3.28 -> 1.36 mm
- net Net-(J4-Pad11): track 1.89 -> 3.36 mm
- net SDA: track 46.2 -> 47.3 mm
- net Net-(U2-ADDR1): track 3.60 -> 3.46 mm, vias 1 -> 0
- added copper zone on B.Cu, net GND
- added copper zone on F.Cu, net GND

Commit message: resolving errors
Connections:
- J4 pad 10: GND -> unconnected-(J4-Pad10)
- R3 pad 1: +3.3V -> +3V3
Routing:
- net Net-(U3-ADDR1): track 1.36 -> 7.24 mm, vias 1 -> 2
- net +3.3V: track 1.02 -> 0.00 mm, vias 1 -> 0
- net +3V3: track 141.3 -> 142.0 mm
- net GND: track 39.8 -> 39.6 mm, vias 14 -> 61
Other:
- board outline added: 35.1 x 55.1 mm

Commit message: clearance errors
Routing:
- net INTERRUPT_F1: track 33.7 -> 31.3 mm
- net GND: track 39.6 -> 37.6 mm
Changed lines of the file:
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@@
       (stroke (width 0.0254) (type solid)) (layer "F.Fab"))
     (pad "1" smd rect (at -2.1971 -0.974999) (size 1.3716 0.4572) (layers "F.Cu" "F.Paste" "F.Mask")
-      (net 13 "SCL") (pinfunction "SCL") (pintype "input"))
+      (net 13 "SCL") (pinfunction "SCL") (pintype "input") (clearance 0.1))
     (pad "2" smd rect (at -2.1971 -0.325001) (size 1.3716 0.4572) (layers "F.Cu" "F.Paste" "F.Mask")
-      (net 10 "INTERRUPT_F2") (pinfunction "ALERT") (pintype "unspecified"))
+      (net 10 "INTERRUPT_F2") (pinfunction "ALERT") (pintype "unspecified") (clearance 0.1))
     (pad "3" smd rect (at -2.1971 0.325001) (size 1.3716 0.4572) (layers "F.Cu" "F.Paste" "F.Mask")
-      (net 19 "Net-(U3-ADDR0)") (pinfunction "ADDR0") (pintype "input"))
+      (net 19 "Net-(U3-ADDR0)") (pinfunction "ADDR0") (pintype "input") (clearance 0.1))
     (pad "4" smd rect (at -2.1971 0.974999) (size 1.3716 0.4572) (layers "F.Cu" "F.Paste" "F.Mask")
       (net 5 "FSR_2") (pinfunction "VIN") (pintype "input"))
     (pad "5" smd rect (at 2.1971 0.974999) (size 1.3716 0.4572) (layers "F.Cu" "F.Paste" "F.Mask")
-      (net 1 "+3V3") (pinfunction "VA") (pintype "power_in"))
+      (net 1 "+3V3") (pinfunction "VA") (pintype "power_in") (clearance 0.1))
     (pad "6" smd rect (at 2.1971 0.325001) (size 1.3716 0.4572) (layers "F.Cu" "F.Paste" "F.Mask")
-      (net 21 "Net-(U3-ADDR1)") (pinfunction "ADDR1") (pintype "input"))
+      (net 21 "Net-(U3-ADDR1)") (pinfunction "ADDR1") (pintype "input") (clearance 0.1))
     (pad "7" smd rect (at 2.1971 -0.325001) (size 1.3716 0.4572) (layers "F.Cu" "F.Paste" "F.Mask")
-      (net 2 "GND") (pinfunction "GND") (pintype "power_in"))
+      (net 2 "GND") (pinfunction "GND") (pintype "power_in") (clearance 0.1))
     (pad "8" smd rect (at 2.1971 -0.974999) (size 1.3716 0.4572) (layers "F.Cu" "F.Paste" "F.Mask")
       (net 14 "SDA") (pinfunction "SDA") (pintype "bidirectional"))
@@
       (stroke (width 0.0254) (type solid)) (layer "F.Fab"))
     (pad "1" smd rect (at -2.1971 -0.974999) (size 1.3716 0.4572) (layers "F.Cu" "F.Paste" "F.Mask")
-      (net 13 "SCL") (pinfunction "SCL") (pintype "input"))
+      (net 13 "SCL") (pinfunction "SCL") (pintype "input") (clearance 0.1))
     (pad "2" smd rect (at -2.1971 -0.325001) (size 1.3716 0.4572) (layers "F.Cu" "F.Paste" "F.Mask")
-      (net 9 "INTERRUPT_F1") (pinfunction "ALERT") (pintype "unspecified"))
+      (net 9 "INTERRUPT_F1") (pinfunction "ALERT") (pintype "unspecified") (clearance 0.1))
     (pad "3" smd rect (at -2.1971 0.325001) (size 1.3716 0.4572) (layers "F.Cu" "F.Paste" "F.Mask")
-      (net 17 "Net-(U2-ADDR0)") (pinfunction "ADDR0") (pintype "input"))
+      (net 17 "Net-(U2-ADDR0)") (pinfunction "ADDR0") (pintype "input") (clearance 0.1))
     (pad "4" smd rect (at -2.1971 0.974999) (size 1.3716 0.4572) (layers "F.Cu" "F.Paste" "F.Mask")
       (net 4 "FSR_1") (pinfunction "VIN") (pintype "input"))
@@
       (net 1 "+3V3") (pinfunction "VA") (pintype "power_in"))
     (pad "6" smd rect (at 2.1971 0.325001) (size 1.3716 0.4572) (layers "F.Cu" "F.Paste" "F.Mask")
-      (net 22 "Net-(U2-ADDR1)") (pinfunction "ADDR1") (pintype "input"))
+      (net 22 "Net-(U2-ADDR1)") (pinfunction "ADDR1") (pintype "input") (clearance 0.1))
     (pad "7" smd rect (at 2.1971 -0.325001) (size 1.3716 0.4572) (layers "F.Cu" "F.Paste" "F.Mask")
-      (net 2 "GND") (pinfunction "GND") (pintype "power_in"))
+      (net 2 "GND") (pinfunction "GND") (pintype "power_in") (clearance 0.1))
     (pad "8" smd rect (at 2.1971 -0.974999) (size 1.3716 0.4572) (layers "F.Cu" "F.Paste" "F.Mask")
       (net 14 "SDA") (pinfunction "SDA") (pintype "bidirectional"))
@@
       (stroke (width 0.0254) (type solid)) (layer "F.Fab"))
     (pad "1" smd rect (at -2.1971 -0.974999) (size 1.3716 0.4572) (layers "F.Cu" "F.Paste" "F.Mask")
-      (net 13 "SCL") (pinfunction "SCL") (pintype "input"))
+      (net 13 "SCL") (pinfunction "SCL") (pintype "input") (clearance 0.1))
     (pad "2" smd rect (at -2.1971 -0.325001) (size 1.3716 0.4572) (layers "F.Cu" "F.Paste" "F.Mask")
-      (net 8 "INTERRUPT_LP") (pinfunction "ALERT") (pintype "unspecified"))
+      (net 8 "INTERRUPT_LP") (pinfunction "ALERT") (pintype "unspecified") (clearance 0.1))
     (pad "3" smd rect (at -2.1971 0.325001) (size 1.3716 0.4572) (layers "F.Cu" "F.Paste" "F.Mask")
-      (net 16 "Net-(U1-ADDR0)") (pinfunction "ADDR0") (pintype "input"))
+      (net 16 "Net-(U1-ADDR0)") (pinfunction "ADDR0") (pintype "input") (clearance 0.1))
     (pad "4" smd rect (at -2.1971 0.974999) (size 1.3716 0.4572) (layers "F.Cu" "F.Paste" "F.Mask")
-      (net 3 "LIN_POT") (pinfunction "VIN") (pintype "input"))
+      (net 3 "LIN_POT") (pinfunction "VIN") (pintype "input") (clearance 0.1))
     (pad "5" smd rect (at 2.1971 0.974999) (size 1.3716 0.4572) (layers "F.Cu" "F.Paste" "F.Mask")
-      (net 1 "+3V3") (pinfunction "VA") (pintype "power_in"))
+      (net 1 "+3V3") (pinfunction "VA") (pintype "power_in") (clearance 0.1))
     (pad "6" smd rect (at 2.1971 0.325001) (size 1.3716 0.4572) (layers "F.Cu" "F.Paste" "F.Mask")
-      (net 20 "Net-(U1-ADDR1)") (pinfunction "ADDR1") (pintype "input"))
+      (net 20 "Net-(U1-ADDR1)") (pinfunction "ADDR1") (pintype "input") (clearance 0.1))
     (pad "7" smd rect (at 2.1971 -0.325001) (size 1.3716 0.4572) (layers "F.Cu" "F.Paste" "F.Mask")
-      (net 2 "GND") (pinfunction "GND") (pintype "power_in"))
+      (net 2 "GND") (pinfunction "GND") (pintype "power_in") (clearance 0.1))
     (pad "8" smd rect (at 2.1971 -0.974999) (size 1.3716 0.4572) (layers "F.Cu" "F.Paste" "F.Mask")
       (net 14 "SDA") (pinfunction "SDA") (pintype "bidirectional"))
@@
       (stroke (width 0.1) (type solid)) (layer "F.Fab"))
     (pad "1" smd roundrect (at -0.51 0 270) (size 0.54 0.64) (layers "F.Cu" "F.Paste" "F.Mask") (roundrect_rratio 0.25)
-      (net 22 "Net-(U2-ADDR1)") (pintype "passive"))
+      (net 22 "Net-(U2-ADDR1)") (pintype "passive") (clearance 0.1))
     (pad "2" smd roundrect (at 0.51 0 270) (size 0.54 0.64) (layers "F.Cu" "F.Paste" "F.Mask") (roundrect_rratio 0.25)
       (net 1 "+3V3") (pintype "passive"))
@@
   (segment (start 35.6108 51.2826) (end 34.159499 51.2826) (width 0.5) (layer "B.Cu") (net 1))
   (segment (start 27.686 57.756099) (end 27.686 58.42) (width 0.5) (layer "B.Cu") (net 1))
-  (segment (start 46.482 39.88) (end 48.288601 39.88) (width 0.25) (layer "F.Cu") (net 2))
   (segment (start 40.64 47.526) (end 40.668 47.498) (width 0.25) (layer "F.Cu") (net 2))
   (segment (start 39.667002 48.188999) (end 38.2651 48.188999) (width 0.25) (layer "F.Cu") (net 2))
@@
   (segment (start 36.068 36.60818) (end 34.694819 35.234999) (width 0.25) (layer "F.Cu") (net 2))
   (segment (start 29.21 51.788) (end 28.982499 51.788) (width 0.25) (layer "F.Cu") (net 2))
-  (segment (start 48.288601 39.88) (end 48.408 39.999399) (width 0.25) (layer "F.Cu") (net 2))
   (segment (start 33.946299 42.633598) (end 34.798 42.633598) (width 0.25) (layer "F.Cu") (net 2))
   (segment (start 29.21 44.45) (end 28.996402 44.663598) (width 0.25) (layer "F.Cu") (net 2))
@@
   (segment (start 48.408 48.749399) (end 44.976601 48.749399) (width 0.25) (layer "F.Cu") (net 8))
   (segment (start 27.6031 46.817399) (end 26.414499 45.628798) (width 0.25) (layer "F.Cu") (net 9))
-  (segment (start 43.307 48.82249) (end 39.46249 52.667) (width 0.25) (layer "F.Cu") (net 9))
-  (segment (start 44.460704 47.499399) (end 43.307 46.345695) (width 0.25) (layer "F.Cu") (net 9))
-  (segment (start 48.408 47.499399) (end 44.460704 47.499399) (width 0.25) (layer "F.Cu") (net 9))
+  (segment (start 34.8817 48.263999) (end 34.8067 48.188999) (width 0.25) (layer "F.Cu") (net 9))
+  (segment (start 44.630091 47.499399) (end 44.47909 47.6504) (width 0.25) (layer "F.Cu") (net 9))
+  (segment (start 48.408 47.499399) (end 44.630091 47.499399) (width 0.25) (layer "F.Cu") (net 9))
   (segment (start 26.414499 45.628798) (end 24.1193 45.628798) (width 0.25) (layer "F.Cu") (net 9))
+  (segment (start 34.8817 51.6457) (end 34.8817 48.263999) (width 0.25) (layer "F.Cu") (net 9))
+  (segment (start 28.9747 48.188999) (end 33.8709 48.188999) (width 0.25) (layer "F.Cu") (net 9))
   (segment (start 39.46249 52.667) (end 35.903 52.667) (width 0.25) (layer "F.Cu") (net 9))
-  (segment (start 28.9747 48.188999) (end 33.8709 48.188999) (width 0.25) (layer "F.Cu") (net 9))
+  (segment (start 44.47909 47.6504) (end 39.46249 52.667) (width 0.25) (layer "F.Cu") (net 9))
+  (segment (start 34.8067 48.188999) (end 33.8709 48.188999) (width 0.25) (layer "F.Cu") (net 9))
+  (segment (start 27.6031 46.817399) (end 28.9747 48.188999) (width 0.25) (layer "F.Cu") (net 9))
   (segment (start 35.903 52.667) (end 34.8817 51.6457) (width 0.25) (layer "F.Cu") (net 9))
-  (segment (start 34.8067 48.188999) (end 33.8709 48.188999) (width 0.25) (layer "F.Cu") (net 9))
-  (segment (start 43.307 46.345695) (end 43.307 48.82249) (width 0.25) (layer "F.Cu") (net 9))
-  (segment (start 27.6031 46.817399) (end 28.9747 48.188999) (width 0.25) (layer "F.Cu") (net 9))
-  (segment (start 34.8817 51.6457) (end 34.8817 48.263999) (width 0.25) (layer "F.Cu") (net 9))
-  (segment (start 34.8817 48.263999) (end 34.8067 48.188999) (width 0.25) (layer "F.Cu") (net 9))
   (segment (start 42.7228 43.7388) (end 33.412121 43.7388) (width 0.25) (layer "F.Cu") (net 10))
   (segment (start 48.386601 46.228) (end 45.212 46.228) (width 0.25) (layer "F.Cu") (net 10))
@@
   (segment (start 27.6031 48.087399) (end 28.354702 48.839001) (width 0.25) (layer "F.Cu") (net 17))
   (segment (start 28.354702 48.839001) (end 33.8709 48.839001) (width 0.25) (layer "F.Cu") (net 17))
+  (segment (start 48.288601 39.88) (end 48.408 39.999399) (width 0.25) (layer "F.Cu") (net 18))
   (segment (start 28.21232 35.885001) (end 29.386221 35.885001) (width 0.25) (layer "F.Cu") (net 19))
   (segment (start 25.997321 38.1) (end 28.21232 35.885001) (width 0.25) (layer "F.Cu") (net 19))

Commit message: 0 errors yay
Routing:
- net FSR_1: track 12.4 -> 15.8 mm
- net GND: track 37.6 -> 40.7 mm
- net FSR_2: track 13.2 -> 16.0 mm
Changed lines of the file:
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@@
   (segment (start 28.956 64.262) (end 27.688 64.262) (width 0.25) (layer "F.Cu") (net 2))
   (segment (start 36.068 36.60818) (end 34.694819 35.234999) (width 0.25) (layer "F.Cu") (net 2))
+  (segment (start 41.1988 60.198) (end 42.8244 58.5724) (width 0.25) (layer "F.Cu") (net 2))
   (segment (start 29.21 51.788) (end 28.982499 51.788) (width 0.25) (layer "F.Cu") (net 2))
   (segment (start 33.946299 42.633598) (end 34.798 42.633598) (width 0.25) (layer "F.Cu") (net 2))
@@
   (segment (start 40.64 47.526) (end 40.330001 47.526) (width 0.25) (layer "F.Cu") (net 2))
   (segment (start 51.308 33.02) (end 51.308 34.949399) (width 0.25) (layer "F.Cu") (net 2))
+  (segment (start 40.386 60.198) (end 41.1988 60.198) (width 0.25) (layer "F.Cu") (net 2))
   (segment (start 28.996402 44.663598) (end 27.5209 44.663598) (width 0.25) (layer "F.Cu") (net 2))
   (segment (start 40.330001 47.526) (end 39.667002 48.188999) (width 0.25) (layer "F.Cu") (net 2))
@@
   (via (at 31.115 44.45) (size 0.8) (drill 0.4) (layers "F.Cu" "B.Cu") (free) (net 2))
   (via (at 38.1 57.785) (size 0.8) (drill 0.4) (layers "F.Cu" "B.Cu") (free) (net 2))
-  (via (at 42.545 57.785) (size 0.8) (drill 0.4) (layers "F.Cu" "B.Cu") (free) (net 2))
+  (via (at 42.8244 58.5724) (size 0.8) (drill 0.4) (layers "F.Cu" "B.Cu") (free) (net 2))
   (via (at 41.91 36.195) (size 0.8) (drill 0.4) (layers "F.Cu" "B.Cu") (free) (net 2))
   (via (at 38.1 55.245) (size 0.8) (drill 0.4) (layers "F.Cu" "B.Cu") (free) (net 2))
@@
   (segment (start 27.94 59.69) (end 25.908 61.722) (width 0.25) (layer "F.Cu") (net 3))
   (segment (start 34.768 61.498) (end 35.9918 61.498) (width 0.25) (layer "F.Cu") (net 3))
+  (segment (start 29.21 50.828) (end 26.19 50.828) (width 0.25) (layer "F.Cu") (net 4))
   (segment (start 25.908 50.546) (end 25.908 52.492299) (width 0.25) (layer "F.Cu") (net 4))
   (segment (start 30.2915 50.8655) (end 30.2915 49.488999) (width 0.25) (layer "F.Cu") (net 4))
+  (segment (start 26.19 50.828) (end 25.908 50.546) (width 0.25) (layer "F.Cu") (net 4))
   (segment (start 30.2915 49.488999) (end 33.8709 49.488999) (width 0.25) (layer "F.Cu") (net 4))
   (segment (start 29.21 50.828) (end 29.21 50.570499) (width 0.25) (layer "F.Cu") (net 4))
@@
   (segment (start 28.448 40.386) (end 28.448 37.47322) (width 0.25) (layer "F.Cu") (net 5))
   (segment (start 28.448 37.47322) (end 29.386221 36.534999) (width 0.25) (layer "F.Cu") (net 5))
+  (segment (start 28.448 40.386) (end 27.94 40.894) (width 0.25) (layer "F.Cu") (net 5))
   (segment (start 25.903 40.894) (end 25.903 43.898598) (width 0.25) (layer "F.Cu") (net 5))
   (segment (start 29.21 42.446) (end 28.448 41.684) (width 0.25) (layer "F.Cu") (net 5))
+  (segment (start 27.94 40.894) (end 25.903 40.894) (width 0.25) (layer "F.Cu") (net 5))
   (segment (start 35.9918 60.198) (end 35.077398 60.198) (width 0.25) (layer "F.Cu") (net 8))
   (segment (start 39.116 57.988202) (end 36.906202 60.198) (width 0.25) (layer "F.Cu") (net 8))
