File: production/ecad/Novel Mechanism 1 Board/Novel Mechanism 1 Board.kicad_sch (KiCad schematic)
At the start: 39 parts, among them J1 Conn_01x02_Socket, J2 Conn_01x02_Socket, J3 Conn_01x02_Socket, J4 0532611271, U1 ADC081C021CIMM/NOPB, U2 ADC081C021CIMM/NOPB, U3 ADC081C021CIMM/NOPB

Commit message: Finished files for Novel Mech 1
Parts:
- C1, C2, C3: LCSC (none) -> C5718966
- C4, C5, C6: LCSC (none) -> C2180807
- C7, C8, C9: LCSC (none) -> C117605
- J4: LCSC (none) -> C17393781
- R1, R13, R2, R3, R4, R5, R9: LCSC (none) -> C881153
- R10, R11, R12: LCSC (none) -> C881209
- R6, R7, R8: LCSC (none) -> C166638
- U1, U2, U3: LCSC (none) -> C206013
Changed lines of the file:
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@@
       (effects (font (size 1.27 1.27)) (justify bottom) hide)
+    )
+    (property "LCSC" "C17393781" (at 264.16 135.89 0)
+      (effects (font (size 1.27 1.27)) hide)
     )
     (pin "1")
@@
       (effects (font (size 1.27 1.27)) hide)
     )
+    (property "LCSC" "C881153" (at 247.65 146.05 0)
+      (effects (font (size 1.27 1.27)) hide)
+    )
     (pin "1")
     (pin "2")
@@
       (effects (font (size 1.27 1.27)) hide)
     )
+    (property "LCSC" "" (at 22.86 19.05 0)
+      (effects (font (size 1.27 1.27)) hide)
+    )
     (instances
       (project "Novel Mechanism 1 Board"
@@
     )
     (property "Datasheet" "~" (at 119.38 170.18 0)
+      (effects (font (size 1.27 1.27)) hide)
+    )
+    (property "LCSC" "C881153" (at 119.38 170.18 0)
       (effects (font (size 1.27 1.27)) hide)
     )
@@
     (property "Datasheet" "ADC081C021CIMM/NOPB" (at 68.58 39.37 0)
       (effects (font (size 1.27 1.27) italic) hide)
+    )
+    (property "LCSC" "C206013" (at 72.39 41.91 0)
+      (effects (font (size 1.27 1.27)) hide)
     )
     (pin "2")
@@
       (effects (font (size 1.27 1.27)) hide)
     )
+    (property "LCSC" "C881209" (at 190.5 95.25 0)
+      (effects (font (size 1.27 1.27)) hide)
+    )
     (pin "2")
     (pin "1")
@@
       (effects (font (size 1.27 1.27)) hide)
     )
+    (property "LCSC" "C881209" (at 190.5 57.15 0)
+      (effects (font (size 1.27 1.27)) hide)
+    )
     (pin "2")
     (pin "1")
@@
       (effects (font (size 1.27 1.27)) hide)
     )
+    (property "LCSC" "C881209" (at 190.5 132.08 0)
+      (effects (font (size 1.27 1.27)) hide)
+    )
     (pin "2")
     (pin "1")
@@
       (effects (font (size 1.27 1.27)) hide)
     )
+    (property "LCSC" "C166638" (at 134.62 152.4 0)
+      (effects (font (size 1.27 1.27)) hide)
+    )
     (pin "1")
     (pin "2")
@@
       (effects (font (size 1.27 1.27)) hide)
     )
+    (property "LCSC" "" (at 195.58 43.18 0)
+      (effects (font (size 1.27 1.27)) hide)
+    )
     (pin "1")
     (pin "2")
@@
     )
     (property "Datasheet" "~" (at 36.83 102.87 0)
+      (effects (font (size 1.27 1.27)) hide)
+    )
+    (property "LCSC" "C2180807" (at 36.83 102.87 0)
       (effects (font (size 1.27 1.27)) hide)
     )
@@
     (property "Datasheet" "ADC081C021CIMM/NOPB" (at 69.85 93.98 0)
       (effects (font (size 1.27 1.27) italic) hide)
+    )
+    (property "LCSC" "C206013" (at 73.66 96.52 0)
+      (effects (font (size 1.27 1.27)) hide)
     )
     (pin "2")
@@
       (effects (font (size 1.27 1.27)) hide)
     )
+    (property "LCSC" "C5718966" (at 25.4 102.87 0)
+      (effects (font (size 1.27 1.27)) hide)
+    )
     (pin "1")
     (pin "2")
@@
       (effects (font (size 1.27 1.27)) hide)
     )
+    (property "LCSC" "C881153" (at 143.51 90.17 0)
+      (effects (font (size 1.27 1.27)) hide)
+    )
     (pin "2")
     (pin "1")
@@
       (effects (font (size 1.27 1.27)) hide)
     )
+    (property "LCSC" "" (at 227.33 88.9 0)
+      (effects (font (size 1.27 1.27)) hide)
+    )
     (pin "1")
     (instances
@@
       (effects (font (size 1.27 1.27)) hide)
     )
+    (property "LCSC" "" (at 227.33 25.4 0)
+      (effects (font (size 1.27 1.27)) hide)
+    )
     (pin "1")
     (instances
@@
       (effects (font (size 1.27 1.27)) hide)
     )
+    (property "LCSC" "C881153" (at 118.11 53.34 0)
+      (effects (font (size 1.27 1.27)) hide)
+    )
     (pin "2")
     (pin "1")
@@
     )
     (property "Datasheet" "~" (at 133.35 36.83 0)
+      (effects (font (size 1.27 1.27)) hide)
+    )
+    (property "LCSC" "C166638" (at 133.35 36.83 0)
       (effects (font (size 1.27 1.27)) hide)
     )
@@
       (effects (font (size 1.27 1.27)) hide)
     )
+    (property "LCSC" "C881153" (at 67.31 57.15 0)
+      (effects (font (size 1.27 1.27)) hide)
+    )
     (pin "2")
     (pin "1")
@@
       (effects (font (size 1.27 1.27)) hide)
     )
+    (property "LCSC" "" (at 45.72 19.05 0)
+      (effects (font (size 1.27 1.27)) hide)
+    )
     (instances
       (project "Novel Mechanism 1 Board"
@@
       (effects (font (size 1.27 1.27)) hide)
     )
+    (property "LCSC" "C117605" (at 62.23 167.64 0)
+      (effects (font (size 1.27 1.27)) hide)
+    )
     (pin "2")
     (pin "1")
@@
     )
     (property "Datasheet" "~" (at 232.41 54.61 0)
+      (effects (font (size 1.27 1.27)) hide)
+    )
+    (property "LCSC" "" (at 227.33 54.61 0)
       (effects (font (size 1.27 1.27)) hide)
     )
@@
       (effects (font (size 1.27 1.27)) hide)
     )
+    (property "LCSC" "C5718966" (at 25.4 165.1 0)
+      (effects (font (size 1.27 1.27)) hide)
+    )
     (pin "1")
     (pin "2")
@@
       (effects (font (size 1.27 1.27)) hide)
     )
+    (property "LCSC" "C881153" (at 71.12 151.13 0)
+      (effects (font (size 1.27 1.27)) hide)
+    )
     (pin "1")
     (pin "2")
@@
     )
     (property "Datasheet" "~" (at 45.72 29.21 0)
+      (effects (font (size 1.27 1.27)) hide)
+    )
+    (property "LCSC" "" (at 45.72 29.21 0)
       (effects (font (size 1.27 1.27)) hide)
     )
@@
     (property "Datasheet" "ADC081C021CIMM/NOPB" (at 69.85 156.21 0)
       (effects (font (size 1.27 1.27) italic) hide)
+    )
+    (property "LCSC" "C206013" (at 73.66 158.75 0)
+      (effects (font (size 1.27 1.27)) hide)
     )
     (pin "2")
@@
       (effects (font (size 1.27 1.27)) hide)
     )
+    (property "LCSC" "C2180807" (at 36.83 165.1 0)
+      (effects (font (size 1.27 1.27)) hide)
+    )
     (pin "1")
     (pin "2")
@@
       (effects (font (size 1.27 1.27)) hide)
     )
+    (property "LCSC" "C5718966" (at 24.13 48.26 0)
+      (effects (font (size 1.27 1.27)) hide)
+    )
     (pin "1")
     (pin "2")
@@
       (effects (font (size 1.27 1.27)) hide)
     )
+    (property "LCSC" "" (at 227.33 40.64 0)
+      (effects (font (size 1.27 1.27)) hide)
+    )
     (pin "1")
     (instances
@@
       (effects (font (size 1.27 1.27)) hide)
     )
+    (property "LCSC" "" (at 227.33 69.85 0)
+      (effects (font (size 1.27 1.27)) hide)
+    )
     (pin "1")
     (instances
@@
       (effects (font (size 1.27 1.27)) hide)
     )
+    (property "LCSC" "C117605" (at 62.23 105.41 0)
+      (effects (font (size 1.27 1.27)) hide)
+    )
     (pin "2")
     (pin "1")
@@
       (effects (font (size 1.27 1.27)) hide)
     )
+    (property "LCSC" "C117605" (at 60.96 50.8 0)
+      (effects (font (size 1.27 1.27)) hide)
+    )
     (pin "2")
     (pin "1")
@@
       (effects (font (size 1.27 1.27)) hide)
     )
+    (property "LCSC" "" (at 195.58 81.28 0)
+      (effects (font (size 1.27 1.27)) hide)
+    )
     (pin "1")
     (pin "2")
@@
       (effects (font (size 1.27 1.27)) hide)
     )
+    (property "LCSC" "C2180807" (at 35.56 48.26 0)
+      (effects (font (size 1.27 1.27)) hide)
+    )
     (pin "1")
     (pin "2")
@@
       (effects (font (size 1.27 1.27)) hide)
     )
+    (property "LCSC" "" (at 260.35 25.4 0)
+      (effects (font (size 1.27 1.27)) hide)
+    )
     (pin "1")
     (instances
@@
       (effects (font (size 1.27 1.27)) hide)
     )
+    (property "LCSC" "" (at 195.58 118.11 0)
+      (effects (font (size 1.27 1.27)) hide)
+    )
     (pin "1")
     (pin "2")
@@
       (effects (font (size 1.27 1.27)) hide)
     )
+    (property "LCSC" "" (at 22.86 29.21 0)
+      (effects (font (size 1.27 1.27)) hide)
+    )
     (instances
       (project "Novel Mechanism 1 Board"
@@
     )
     (property "Datasheet" "~" (at 134.62 90.17 0)
+      (effects (font (size 1.27 1.27)) hide)
+    )
+    (property "LCSC" "C166638" (at 134.62 90.17 0)
       (effects (font (size 1.27 1.27)) hide)
     )
@@
       (effects (font (size 1.27 1.27)) hide)
     )
+    (property "LCSC" "C881153" (at 69.85 110.49 0)
+      (effects (font (size 1.27 1.27)) hide)
+    )
