File: production/ecad/Novel Mechanism 2 Board/Novel Mechanism 2 Board.kicad_sch (KiCad schematic)
At the start: 16 parts, among them J1 1755736, J2 1755736, J4 Conn_01x12_Pin, U1 L9958SBTR, U2 TMCS1108A4BQDRQ1

Commit message: added correct connector
Parts:
- removed J4: Conn_01x12_Pin, symbol Connector:Conn_01x12_Pin
- added J3: 0532611271, 0532611271:MOLEX_0532611271, symbol 4xxx:0532611271
- added R3: 10k, Resistor_SMD:RES_0603, symbol Device:R
Connections:
- net +5V: now also J3.1
- net AOUT: now also J3.7
- net ChipSel: now also J3.6
- net DET: now also J3.11, R3.2
- net Direction: now also J3.5
- net Disable: now also J3.2
- net Enable: now also J3.3
- net GND: now also C2.2, C3.2
- net PWM: now also J3.4
- net SCK: now also J3.8
- net SI: now also J3.9
- net SO: now also J3.10
- new net: J3.12, R3.1
- no-connect marks 1 -> 0

Commit message: added resistor divider at aout to fit within microcontroller adc range
Parts:
- added R4: 10k, Resistor_SMD:RES_0603, symbol Device:R
- added R5: 50k, Resistor_SMD:RES_0603, symbol Device:R
Connections:
- net AOUT: now also R4.2, R5.1; no longer U2.7 (VOUT)
- net GND: now also R5.2
- new net: R4.1, U2.7 (VOUT)
Changed lines of the file:
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@@
   (junction (at 93.98 41.91) (diameter 0) (color 0 0 0 0)
   )
+  (junction (at 182.245 56.515) (diameter 0) (color 0 0 0 0)
+  )
   (junction (at 102.87 76.2) (diameter 0) (color 0 0 0 0)
   )
@@
     (stroke (width 0) (type default))
   )
-  (wire (pts (xy 165.735 47.625) (xy 173.355 47.625))
+  (wire (pts (xy 165.735 47.625) (xy 182.245 47.625))
     (stroke (width 0) (type default))
   )
@@
     (stroke (width 0) (type default))
   )
+  (wire (pts (xy 182.245 56.515) (xy 182.245 55.245))
+    (stroke (width 0) (type default))
+  )
   (wire (pts (xy 23.495 61.595) (xy 35.56 61.595))
     (stroke (width 0) (type default))
@@
     (stroke (width 0) (type default))
   )
+  (wire (pts (xy 182.245 56.515) (xy 193.675 56.515))
+    (stroke (width 0) (type default))
+  )
   (wire (pts (xy 38.735 136.525) (xy 29.845 136.525))
     (stroke (width 0) (type default))
@@
     (stroke (width 0) (type default))
   )
+  (wire (pts (xy 182.245 57.15) (xy 182.245 56.515))
+    (stroke (width 0) (type default))
+  )
   (wire (pts (xy 38.735 128.905) (xy 29.845 128.905))
     (stroke (width 0) (type default))
@@
     (stroke (width 0) (type default))
   )
-  (label "AOUT" (at 173.355 47.625 180) (fields_autoplaced)
+  (label "AOUT" (at 193.675 56.515 180) (fields_autoplaced)
     (effects (font (size 1.27 1.27)) (justify right bottom))
   )
@@
         (path "/148ef552-79ac-46c4-a436-ee743f083e73"
           (reference "#PWR09") (unit 1)
+        )
+      )
+    )
+  )
+  (symbol (lib_id "Device:R") (at 182.245 60.96 0) (unit 1)
+    (in_bom yes) (on_board yes) (dnp no) (fields_autoplaced)
+    (property "Reference" "R5" (at 184.15 59.69 0)
+      (effects (font (size 1.27 1.27)) (justify left))
+    )
+    (property "Value" "50k" (at 184.15 62.23 0)
+      (effects (font (size 1.27 1.27)) (justify left))
+    )
+    (property "Footprint" "Resistor_SMD:RES_0603" (at 180.467 60.96 90)
+      (effects (font (size 1.27 1.27)) hide)
+    )
+    (property "Datasheet" "~" (at 182.245 60.96 0)
+      (effects (font (size 1.27 1.27)) hide)
+    )
+    (pin "2")
+    (pin "1")
+    (instances
+      (project "Novel Mechanism 2 Board"
+        (path "/148ef552-79ac-46c4-a436-ee743f083e73"
+          (reference "R5") (unit 1)
         )
       )
@@
     )
   )
+  (symbol (lib_id "Device:R") (at 182.245 51.435 0) (unit 1)
+    (in_bom yes) (on_board yes) (dnp no) (fields_autoplaced)
+    (property "Reference" "R4" (at 184.785 50.165 0)
+      (effects (font (size 1.27 1.27)) (justify left))
+    )
+    (property "Value" "10k" (at 184.785 52.705 0)
+      (effects (font (size 1.27 1.27)) (justify left))
+    )
+    (property "Footprint" "Resistor_SMD:RES_0603" (at 180.467 51.435 90)
+      (effects (font (size 1.27 1.27)) hide)
+    )
+    (property "Datasheet" "~" (at 182.245 51.435 0)
+      (effects (font (size 1.27 1.27)) hide)
+    )
+    (pin "2")
+    (pin "1")
+    (instances
+      (project "Novel Mechanism 2 Board"
+        (path "/148ef552-79ac-46c4-a436-ee743f083e73"
+          (reference "R4") (unit 1)
+        )
+      )
+    )
+  )
   (symbol (lib_id "power:+5V") (at 23.495 59.69 0) (unit 1)
     (in_bom yes) (on_board yes) (dnp no) (fields_autoplaced)
@@
         )
       )
+    )
+  )
+  (symbol (lib_id "power:GND") (at 182.245 64.77 0) (unit 1)
+    (in_bom yes) (on_board yes) (dnp no) (fields_autoplaced)
+    (property "Reference" "#PWR02" (at 182.245 71.12 0)
+      (effects (font (size 1.27 1.27)) hide)
+    )
+    (property "Value" "GND" (at 182.245 69.215 0)
+      (effects (font (size 1.27 1.27)))
+    )
+    (property "Footprint" "" (at 182.245 64.77 0)
+      (effects (font (size 1.27 1.27)) hide)
+    )
+    (property "Datasheet" "" (at 182.245 64.77 0)
+      (effects (font (size 1.27 1.27)) hide)
+    )
+    (pin "1")
+    (instances
+      (project "Novel Mechanism 2 Board"
+        (path "/148ef552-79ac-46c4-a436-ee743f083e73"
+          (reference "#PWR02") (unit 1)
+        )
+      )

Commit message: updated footprint
Parts:
- J3: footprint 0532611271:MOLEX_0532611271 -> Connector:MOLEX_0532611271
Changed lines of the file:
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@@
       (effects (font (size 1.27 1.27)) (justify left))
     )
-    (property "Footprint" "0532611271:MOLEX_0532611271" (at 48.895 139.065 0)
+    (property "Footprint" "Connector:MOLEX_0532611271" (at 48.895 139.065 0)
       (effects (font (size 1.27 1.27)) (justify bottom) hide)
     )

Commit message: signal routing complete!
Connections:
- net +15V: no longer U1.13 (VS)
- net +5V: no longer U1.16 (VDD)
- net ChipSel: no longer U1.3 (CS)
- net Direction: no longer U1.5 (DIR)
- net Disable: no longer U1.7 (DI)
- net Enable: no longer U1.9 (EN)
- net GND: now also U1.12 (REXT); no longer U1.1 (GND), U1.17 (EXP), U1.8 (PGND)
- net PWM: no longer U1.11 (PWM)
- net SCK: no longer U1.15 (SCK)
- net SI: no longer U1.14 (SI)
- net SO: no longer U1.2 (SO)
- net at C7.1, J2.1: no longer U1.10 (OUT2)
- net at C6.1, U2.1 (IN+), U2.2 (IN+__1): no longer U1.6 (OUT1)
- net at C1.2: no longer U1.4 (CP)
- net at R2.1: now also U1.17 (EXP); no longer U1.12 (REXT)
Changed lines of the file:
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@@
     )
   )
-  (symbol (lib_id "L9958SBTR:L9958SBTR") (at 81.915 81.28 0) (unit 1)
+  (symbol (lib_id "L9958SBTR:L9958SBTR") (at 81.915 81.28 0) (mirror y) (unit 1)
     (in_bom yes) (on_board yes) (dnp no)
-    (property "Reference" "U1" (at 82.55 78.74 0)
+    (property "Reference" "U1" (at 81.28 78.74 0)
       (effects (font (size 1.27 1.27)))
     )
-    (property "Value" "L9958SBTR" (at 82.55 81.28 0)
+    (property "Value" "L9958SBTR" (at 81.28 81.28 0)
       (effects (font (size 1.27 1.27)))
     )

Commit message: routing complete - preteardrops
Connections:
- net +15V: now also U1.13 (VS)
- net +5V: now also U1.16 (VDD)
- net ChipSel: now also U1.3 (CS)
- net Direction: now also U1.5 (DIR)
- net Disable: now also U1.7 (DI)
- net Enable: now also U1.9 (EN)
- net GND: now also U1.1 (GND), U1.17 (EXP), U1.8 (PGND); no longer U1.12 (REXT)
- net PWM: now also U1.11 (PWM)
- net SCK: now also U1.15 (SCK)
- net SI: now also U1.14 (SI)
- net SO: now also U1.2 (SO)
- net at C7.1, J2.1: now also U1.10 (OUT2)
- net at U2.1 (IN+), U2.2 (IN+__1): now also J2.2; no longer C6.1
- net at U2.3 (IN-), U2.4 (IN-__1): now also C6.1, U1.6 (OUT1); no longer J2.2
- net at C1.2: now also U1.4 (CP)
- net at R2.1: now also U1.12 (REXT); no longer U1.17 (EXP)
Changed lines of the file:
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@@
   (junction (at 78.105 31.115) (diameter 0) (color 0 0 0 0)
   )
+  (junction (at 88.265 31.115) (diameter 0) (color 0 0 0 0)
+  )
+  (junction (at 93.98 41.91) (diameter 0) (color 0 0 0 0)
+  )
+  (junction (at 102.87 62.23) (diameter 0) (color 0 0 0 0)
+  )
+  (junction (at 135.255 47.625) (diameter 0) (color 0 0 0 0)
+  )
+  (junction (at 182.245 56.515) (diameter 0) (color 0 0 0 0)
+  )
+  (junction (at 102.87 76.2) (diameter 0) (color 0 0 0 0)
+  )
+  (junction (at 23.495 71.12) (diameter 0) (color 0 0 0 0)
+  )
+  (junction (at 101.6 102.87) (diameter 0) (color 0 0 0 0)
+  )
+  (junction (at 101.6 96.52) (diameter 0) (color 0 0 0 0)
+  )
+  (junction (at 93.98 31.115) (diameter 0) (color 0 0 0 0)
+  )
+  (junction (at 23.495 61.595) (diameter 0) (color 0 0 0 0)
+  )
   (junction (at 135.255 55.245) (diameter 0) (color 0 0 0 0)
   )
-  (junction (at 88.265 31.115) (diameter 0) (color 0 0 0 0)
-  )
-  (junction (at 93.98 41.91) (diameter 0) (color 0 0 0 0)
-  )
-  (junction (at 182.245 56.515) (diameter 0) (color 0 0 0 0)
-  )
-  (junction (at 102.87 76.2) (diameter 0) (color 0 0 0 0)
-  )
-  (junction (at 23.495 71.12) (diameter 0) (color 0 0 0 0)
-  )
-  (junction (at 101.6 102.87) (diameter 0) (color 0 0 0 0)
-  )
-  (junction (at 102.87 62.23) (diameter 0) (color 0 0 0 0)
-  )
-  (junction (at 101.6 96.52) (diameter 0) (color 0 0 0 0)
-  )
-  (junction (at 93.98 31.115) (diameter 0) (color 0 0 0 0)
-  )
-  (junction (at 23.495 61.595) (diameter 0) (color 0 0 0 0)
-  )
   (junction (at 58.42 31.115) (diameter 0) (color 0 0 0 0)
   )
   (junction (at 23.495 59.69) (diameter 0) (color 0 0 0 0)
   )
-  (junction (at 135.255 47.625) (diameter 0) (color 0 0 0 0)
-  )
   (wire (pts (xy 15.875 141.605) (xy 19.05 141.605))
     (stroke (width 0) (type default))
   )
+  (wire (pts (xy 102.87 55.245) (xy 102.87 62.23))
+    (stroke (width 0) (type default))
+  )
   (wire (pts (xy 38.735 141.605) (xy 29.845 141.605))
     (stroke (width 0) (type default))
@@
     (stroke (width 0) (type default))
   )
-  (wire (pts (xy 102.87 47.625) (xy 135.255 47.625))
-    (stroke (width 0) (type default))
-  )
   (wire (pts (xy 66.675 71.12) (xy 59.055 71.12))
     (stroke (width 0) (type default))
   )
+  (wire (pts (xy 104.775 31.115) (xy 104.775 33.02))
+    (stroke (width 0) (type default))
+  )
+  (wire (pts (xy 93.98 31.115) (xy 93.98 33.02))
+    (stroke (width 0) (type default))
+  )
+  (wire (pts (xy 102.87 55.245) (xy 135.255 55.245))
+    (stroke (width 0) (type default))
+  )
+  (wire (pts (xy 51.435 67.31) (xy 51.435 69.215))
+    (stroke (width 0) (type default))
+  )
+  (wire (pts (xy 38.735 144.145) (xy 29.845 144.145))
+    (stroke (width 0) (type default))
+  )
   (wire (pts (xy 97.155 96.52) (xy 101.6 96.52))
     (stroke (width 0) (type default))
   )
-  (wire (pts (xy 104.775 31.115) (xy 104.775 33.02))
-    (stroke (width 0) (type default))
-  )
-  (wire (pts (xy 93.98 31.115) (xy 93.98 33.02))
-    (stroke (width 0) (type default))
-  )
-  (wire (pts (xy 51.435 67.31) (xy 51.435 69.215))
-    (stroke (width 0) (type default))
-  )
-  (wire (pts (xy 38.735 144.145) (xy 29.845 144.145))
-    (stroke (width 0) (type default))
-  )
   (wire (pts (xy 101.6 96.52) (xy 101.6 102.87))
     (stroke (width 0) (type default))
@@
     (stroke (width 0) (type default))
   )
-  (wire (pts (xy 130.81 55.245) (xy 130.81 71.12))
+  (wire (pts (xy 130.81 47.625) (xy 130.81 71.12))
     (stroke (width 0) (type default))
   )
@@
     (stroke (width 0) (type default))
   )
-  (wire (pts (xy 102.87 62.23) (xy 102.87 47.625))
-    (stroke (width 0) (type default))
-  )
   (wire (pts (xy 29.845 139.065) (xy 38.735 139.065))
     (stroke (width 0) (type default))
@@
     (stroke (width 0) (type default))
   )
-  (wire (pts (xy 135.255 55.245) (xy 130.81 55.245))
-    (stroke (width 0) (type default))
-  )
   (wire (pts (xy 102.87 76.2) (xy 190.5 76.2))
     (stroke (width 0) (type default))
@@
   )
   (wire (pts (xy 59.055 95.25) (xy 66.675 95.25))
+    (stroke (width 0) (type default))
+  )
+  (wire (pts (xy 130.81 47.625) (xy 135.255 47.625))
     (stroke (width 0) (type default))
   )
@@
     )
   )
-  (symbol (lib_id "L9958SBTR:L9958SBTR") (at 81.915 81.28 0) (mirror y) (unit 1)
+  (symbol (lib_id "L9958SBTR:L9958SBTR") (at 81.915 81.28 0) (unit 1)
     (in_bom yes) (on_board yes) (dnp no)
-    (property "Reference" "U1" (at 81.28 78.74 0)
-      (effects (font (size 1.27 1.27)))
-    )
-    (property "Value" "L9958SBTR" (at 81.28 81.28 0)
-      (effects (font (size 1.27 1.27)))
-    )
+    (property "Reference" "U1" (at 82.55 78.74 0)
+      (effects (font (size 1.27 1.27)))
+    )
+    (property "Value" "L9958SBTR" (at 82.55 81.28 0)
+      (effects (font (size 1.27 1.27)))
+    )

Commit message: added mounting holes
Parts:
- added H2, H3, H4: MountingHole, MountingHole:MountingHole_3.2mm_M3, symbol Mechanical:MountingHole
Changed lines of the file:
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@@
+    )
+  )
+  (symbol (lib_id "Mechanical:MountingHole") (at 133.35 93.98 0) (unit 1)
+    (in_bom yes) (on_board yes) (dnp no) (fields_autoplaced)
+    (property "Reference" "H2" (at 135.89 92.71 0)
+      (effects (font (size 1.27 1.27)) (justify left))
+    )
+    (property "Value" "MountingHole" (at 135.89 95.25 0)
+      (effects (font (size 1.27 1.27)) (justify left))
+    )
+    (property "Footprint" "MountingHole:MountingHole_3.2mm_M3" (at 133.35 93.98 0)
+      (effects (font (size 1.27 1.27)) hide)
+    )
+    (property "Datasheet" "~" (at 133.35 93.98 0)
+      (effects (font (size 1.27 1.27)) hide)
+    )
+    (instances
+      (project "Novel Mechanism 2 Board"
+        (path "/148ef552-79ac-46c4-a436-ee743f083e73"
+          (reference "H2") (unit 1)
+        )
+      )
+    )
+  )
+  (symbol (lib_id "Mechanical:MountingHole") (at 133.35 106.045 0) (unit 1)
+    (in_bom yes) (on_board yes) (dnp no) (fields_autoplaced)
+    (property "Reference" "H4" (at 135.89 104.775 0)
+      (effects (font (size 1.27 1.27)) (justify left))
+    )
+    (property "Value" "MountingHole" (at 135.89 107.315 0)
+      (effects (font (size 1.27 1.27)) (justify left))
+    )
+    (property "Footprint" "MountingHole:MountingHole_3.2mm_M3" (at 133.35 106.045 0)
+      (effects (font (size 1.27 1.27)) hide)
+    )
+    (property "Datasheet" "~" (at 133.35 106.045 0)
+      (effects (font (size 1.27 1.27)) hide)
+    )
+    (instances
+      (project "Novel Mechanism 2 Board"
+        (path "/148ef552-79ac-46c4-a436-ee743f083e73"
+          (reference "H4") (unit 1)
+        )
+      )
     )
   )
@@
         )
       )
+    )
+  )
+  (symbol (lib_id "Mechanical:MountingHole") (at 133.35 100.33 0) (unit 1)
+    (in_bom yes) (on_board yes) (dnp no) (fields_autoplaced)
+    (property "Reference" "H3" (at 135.89 99.06 0)
+      (effects (font (size 1.27 1.27)) (justify left))
+    )
+    (property "Value" "MountingHole" (at 135.89 101.6 0)
+      (effects (font (size 1.27 1.27)) (justify left))
+    )
+    (property "Footprint" "MountingHole:MountingHole_3.2mm_M3" (at 133.35 100.33 0)
+      (effects (font (size 1.27 1.27)) hide)
+    )
+    (property "Datasheet" "~" (at 133.35 100.33 0)
+      (effects (font (size 1.27 1.27)) hide)
+    )
+    (instances
+      (project "Novel Mechanism 2 Board"
+        (path "/148ef552-79ac-46c4-a436-ee743f083e73"
+          (reference "H3") (unit 1)
+        )
+      )

Commit message: final board edits
Parts:
- renumbered H3 to H1, H4 to H3
Changed lines of the file:
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@@
   (symbol (lib_id "Mechanical:MountingHole") (at 133.35 106.045 0) (unit 1)
     (in_bom yes) (on_board yes) (dnp no) (fields_autoplaced)
-    (property "Reference" "H4" (at 135.89 104.775 0)
+    (property "Reference" "H3" (at 135.89 104.775 0)
       (effects (font (size 1.27 1.27)) (justify left))
     )
@@
       (project "Novel Mechanism 2 Board"
         (path "/148ef552-79ac-46c4-a436-ee743f083e73"
-          (reference "H4") (unit 1)
+          (reference "H3") (unit 1)
         )
       )
@@
   (symbol (lib_id "Mechanical:MountingHole") (at 133.35 100.33 0) (unit 1)
     (in_bom yes) (on_board yes) (dnp no) (fields_autoplaced)
-    (property "Reference" "H3" (at 135.89 99.06 0)
+    (property "Reference" "H1" (at 135.89 99.06 0)
       (effects (font (size 1.27 1.27)) (justify left))
     )
@@
       (project "Novel Mechanism 2 Board"
         (path "/148ef552-79ac-46c4-a436-ee743f083e73"
-          (reference "H3") (unit 1)
-        )
-      )
+          (reference "H1") (unit 1)
+        )
+      )

Commit message: added jlc part numbers
Parts:
- C1, C4: LCSC (none) -> C385964
- C2: LCSC (none) -> C1498019
- C3: LCSC (none) -> C2167154
- C5: LCSC (none) -> C2162961
- C6, C7: LCSC (none) -> C161232
- CR1: LCSC (none) -> C1665786
- CR2: LCSC (none) -> STTH4R02U
- J1, J2: LCSC (none) -> C480503
- J3: LCSC (none) -> C277633
- R1: LCSC (none) -> C441928
- R2, R3, R4: LCSC (none) -> C441927
- R5: LCSC (none) -> C445844
- U1: LCSC (none) -> C2150675
- U2: LCSC (none) -> C3684247
Changed lines of the file:
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@@
+      (effects (font (size 1.27 1.27)) hide)
+    )
+    (property "LCSC" "C161232" (at 102.87 80.01 0)
       (effects (font (size 1.27 1.27)) hide)
     )
@@
     (property "E_MAX" "6.19" (at 150.495 50.165 0)
       (effects (font (size 1.27 1.27)) (justify bottom) hide)
+    )
+    (property "LCSC" "C3684247" (at 150.495 50.165 0)
+      (effects (font (size 1.27 1.27)) hide)
     )
     (pin "4")
@@
       (effects (font (size 1.27 1.27)) hide)
     )
+    (property "LCSC" "C385964" (at 78.105 36.83 0)
+      (effects (font (size 1.27 1.27)) hide)
+    )
     (pin "2")
     (pin "1")
@@
       (effects (font (size 1.27 1.27)) hide)
     )
+    (property "LCSC" "C2162961" (at 35.56 66.675 0)
+      (effects (font (size 1.27 1.27)) hide)
+    )
     (pin "2")
     (pin "1")
@@
       (effects (font (size 1.27 1.27)) hide)
     )
+    (property "LCSC" "C441927" (at 19.05 145.415 0)
+      (effects (font (size 1.27 1.27)) hide)
+    )
     (pin "2")
     (pin "1")
@@
     )
     (property "Datasheet" "~" (at 182.245 60.96 0)
+      (effects (font (size 1.27 1.27)) hide)
+    )
+    (property "LCSC" "C445844" (at 182.245 60.96 0)
       (effects (font (size 1.27 1.27)) hide)
     )
@@
     (property "STANDARD" "IPC-7351B" (at 81.915 81.28 0)
       (effects (font (size 1.27 1.27)) (justify bottom) hide)
+    )
+    (property "LCSC" "C2150675" (at 81.915 81.28 0)
+      (effects (font (size 1.27 1.27)) hide)
     )
     (pin "12")
@@
       (effects (font (size 1.27 1.27)) hide)
     )
+    (property "LCSC" "C441927" (at 182.245 51.435 0)
+      (effects (font (size 1.27 1.27)) hide)
+    )
     (pin "2")
     (pin "1")
@@
     (property "STANDARD" "Manufacturer Recommendations" (at 48.895 139.065 0)
       (effects (font (size 1.27 1.27)) (justify bottom) hide)
+    )
+    (property "LCSC" "C277633" (at 48.895 139.065 0)
+      (effects (font (size 1.27 1.27)) hide)
     )
     (pin "5")
@@
       (effects (font (size 1.27 1.27)) (justify bottom) hide)
     )
+    (property "LCSC" "C480503" (at 28.575 33.655 0)
+      (effects (font (size 1.27 1.27)) hide)
+    )
     (pin "1")
     (pin "2")
@@
       (effects (font (size 1.27 1.27)) hide)
     )
+    (property "LCSC" "C161232" (at 102.87 66.04 0)
+      (effects (font (size 1.27 1.27)) hide)
+    )
     (pin "2")
     (pin "1")
@@
       (effects (font (size 1.27 1.27)) hide)
     )
+    (property "LCSC" "" (at 133.35 93.98 0)
+      (effects (font (size 1.27 1.27)) hide)
+    )
     (instances
       (project "Novel Mechanism 2 Board"
@@
       (effects (font (size 1.27 1.27)) hide)
     )
+    (property "LCSC" "" (at 133.35 106.045 0)
+      (effects (font (size 1.27 1.27)) hide)
+    )
     (instances
       (project "Novel Mechanism 2 Board"
@@
       (effects (font (size 1.27 1.27)) hide)
     )
+    (property "LCSC" "C441927" (at 59.055 106.68 0)
+      (effects (font (size 1.27 1.27)) hide)
+    )
     (pin "2")
     (pin "1")
@@
       (effects (font (size 1.27 1.27)) hide)
     )
+    (property "LCSC" "C1498019" (at 93.98 36.83 0)
+      (effects (font (size 1.27 1.27)) hide)
+    )
     (pin "2")
     (pin "1")
@@
     )
     (property "Datasheet" "~" (at 23.495 66.675 0)
+      (effects (font (size 1.27 1.27)) hide)
+    )
+    (property "LCSC" "C385964" (at 23.495 66.675 0)
       (effects (font (size 1.27 1.27)) hide)
     )
@@
       (effects (font (size 1.27 1.27) italic) hide)
     )
+    (property "LCSC" "STTH4R02U" (at 52.07 31.115 0)
+      (effects (font (size 1.27 1.27)) hide)
+    )
     (pin "2")
     (pin "1")
@@
       (effects (font (size 1.27 1.27)) hide)
     )
+    (property "LCSC" "C2167154" (at 104.775 36.83 0)
+      (effects (font (size 1.27 1.27)) hide)
+    )
     (pin "2")
     (pin "1")
@@
     )
     (property "Datasheet" "~" (at 133.35 100.33 0)
+      (effects (font (size 1.27 1.27)) hide)
+    )
+    (property "LCSC" "" (at 133.35 100.33 0)
       (effects (font (size 1.27 1.27)) hide)
     )
@@
     (property "Datasheet" "BZW50-27B" (at 58.42 31.115 0)
       (effects (font (size 1.27 1.27) italic) hide)
+    )
+    (property "LCSC" "C1665786" (at 58.42 31.115 0)
+      (effects (font (size 1.27 1.27)) hide)
     )
     (pin "2")
@@
       (effects (font (size 1.27 1.27)) (justify bottom) hide)
     )
+    (property "LCSC" "C480503" (at 198.12 71.12 0)
+      (effects (font (size 1.27 1.27)) hide)
+    )
     (pin "1")
     (pin "2")
@@
       (effects (font (size 1.27 1.27)) hide)
     )
+    (property "LCSC" "C441928" (at 51.435 73.025 0)
+      (effects (font (size 1.27 1.27)) hide)
+    )
